File: Hardware/4-20mAConverter.kicad_sch (KiCad schematic)
At the start: 26 parts, among them J7 Screw_Terminal, Q3 NPN, U5 LM317_TO-252, U6 LM324, U7 TL431

Commit message: add R0603 footprint
Parts:
- D3: value D_Diode -> D_Schottky
Changed lines of the file:
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@@
   (symbol (lib_id "power:GND") (at 115.57 53.975 0) (unit 1)
     (in_bom yes) (on_board yes)
-    (property "Reference" "#PWR?" (id 0) (at 115.57 60.325 0)
+    (property "Reference" "#PWR0249" (id 0) (at 115.57 60.325 0)
       (effects (font (size 1.27 1.27)) hide)
     )
@@
   (symbol (lib_id "power:GND") (at 77.47 97.79 0) (unit 1)
     (in_bom yes) (on_board yes)
-    (property "Reference" "#PWR?" (id 0) (at 77.47 104.14 0)
+    (property "Reference" "#PWR0244" (id 0) (at 77.47 104.14 0)
       (effects (font (size 1.27 1.27)) hide)
     )
@@
   (symbol (lib_id "power:GND") (at 92.71 97.155 0) (unit 1)
     (in_bom yes) (on_board yes)
-    (property "Reference" "#PWR?" (id 0) (at 92.71 103.505 0)
+    (property "Reference" "#PWR0246" (id 0) (at 92.71 103.505 0)
       (effects (font (size 1.27 1.27)) hide)
     )
@@
   (symbol (lib_id "power:VCC") (at 26.67 66.04 0) (unit 1)
     (in_bom yes) (on_board yes) (fields_autoplaced)
-    (property "Reference" "#PWR?" (id 0) (at 26.67 69.85 0)
+    (property "Reference" "#PWR0254" (id 0) (at 26.67 69.85 0)
       (effects (font (size 1.27 1.27)) hide)
     )
@@
   (symbol (lib_id "power:GND") (at 63.5 97.79 0) (unit 1)
     (in_bom yes) (on_board yes)
-    (property "Reference" "#PWR?" (id 0) (at 63.5 104.14 0)
+    (property "Reference" "#PWR0245" (id 0) (at 63.5 104.14 0)
       (effects (font (size 1.27 1.27)) hide)
     )
@@
   (symbol (lib_id "power:GND") (at 92.075 53.975 0) (unit 1)
     (in_bom yes) (on_board yes) (fields_autoplaced)
-    (property "Reference" "#PWR?" (id 0) (at 92.075 60.325 0)
+    (property "Reference" "#PWR0248" (id 0) (at 92.075 60.325 0)
       (effects (font (size 1.27 1.27)) hide)
     )
@@
   (symbol (lib_id "power:GND") (at 145.415 75.565 0) (unit 1)
     (in_bom yes) (on_board yes)
-    (property "Reference" "#PWR?" (id 0) (at 145.415 81.915 0)
+    (property "Reference" "#PWR0252" (id 0) (at 145.415 81.915 0)
       (effects (font (size 1.27 1.27)) hide)
     )
@@
   (symbol (lib_id "power:VCC") (at 198.12 104.14 0) (unit 1)
     (in_bom yes) (on_board yes) (fields_autoplaced)
-    (property "Reference" "#PWR?" (id 0) (at 198.12 107.95 0)
+    (property "Reference" "#PWR0256" (id 0) (at 198.12 107.95 0)
       (effects (font (size 1.27 1.27)) hide)
     )
@@
   (symbol (lib_id "power:GND") (at 198.12 118.11 0) (unit 1)
     (in_bom yes) (on_board yes)
-    (property "Reference" "#PWR?" (id 0) (at 198.12 124.46 0)
+    (property "Reference" "#PWR0255" (id 0) (at 198.12 124.46 0)
       (effects (font (size 1.27 1.27)) hide)
     )
@@
   (symbol (lib_id "power:GND") (at 26.67 102.235 0) (unit 1)
     (in_bom yes) (on_board yes) (fields_autoplaced)
-    (property "Reference" "#PWR?" (id 0) (at 26.67 108.585 0)
+    (property "Reference" "#PWR0250" (id 0) (at 26.67 108.585 0)
       (effects (font (size 1.27 1.27)) hide)
     )
@@
   (symbol (lib_id "power:GND") (at 152.4 75.565 0) (unit 1)
     (in_bom yes) (on_board yes)
-    (property "Reference" "#PWR?" (id 0) (at 152.4 81.915 0)
+    (property "Reference" "#PWR0253" (id 0) (at 152.4 81.915 0)
       (effects (font (size 1.27 1.27)) hide)
     )
@@
     (in_bom yes) (on_board yes) (fields_autoplaced)
     (property "Reference" "D3" (id 0) (at 35.56 66.04 0))
-    (property "Value" "D_Diode" (id 1) (at 35.56 68.58 0))
+    (property "Value" "D_Schottky" (id 1) (at 35.56 68.58 0))
     (property "Footprint" "IVS_FOOTPRINTS:D_SMA" (id 2) (at 36.83 67.31 0)
       (effects (font (size 1.27 1.27)) hide)
@@
   (symbol (lib_id "power:GND") (at 160.655 107.315 0) (unit 1)
     (in_bom yes) (on_board yes)
-    (property "Reference" "#PWR?" (id 0) (at 160.655 113.665 0)
+    (property "Reference" "#PWR0251" (id 0) (at 160.655 113.665 0)
       (effects (font (size 1.27 1.27)) hide)
     )
@@
   (symbol (lib_id "power:GND") (at 111.125 97.79 0) (unit 1)
     (in_bom yes) (on_board yes)
-    (property "Reference" "#PWR?" (id 0) (at 111.125 104.14 0)
-      (effects (font (size 1.27 1.27)) hide)
-    )
+    (property "Reference" "#PWR0247" (id 0) (at 111.125 104.14 0)
+      (effects (font (size 1.27 1.27)) hide)
+    )

Commit message: fix name and move pin 74hc165
Parts:
- RV2, RV3: footprint (none) -> IVS_FOOTPRINTS:Potentiometer_Bourns_TC33X_Vertical
Changed lines of the file:
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@@
       (effects (font (size 1.27 1.27)) (justify right))
     )
-    (property "Footprint" "" (id 2) (at 115.57 48.895 0)
+    (property "Footprint" "IVS_FOOTPRINTS:Potentiometer_Bourns_TC33X_Vertical" (id 2) (at 115.57 48.895 0)
       (effects (font (size 1.27 1.27)) hide)
     )
@@
       (effects (font (size 1.27 1.27)) (justify right))
     )
-    (property "Footprint" "" (id 2) (at 111.125 80.645 0)
+    (property "Footprint" "IVS_FOOTPRINTS:Potentiometer_Bourns_TC33X_Vertical" (id 2) (at 111.125 80.645 0)
       (effects (font (size 1.27 1.27)) hide)
     )

Commit message: fix MCP41010, fix symbol output header
Parts:
- renumbered C33 to C32, D3 to D24, J7 to J22, LE2 to LE1, LE3 to LE2, Q3 to Q17, R30 to R100, R32 to R101, R33 to R102, R34 to R103, R40 to R104, R39 to R105, R35 to R106, R37 to R107, R36 to R108, R38 to R109, R26 to R95, R27 to R96, R28 to R97, R29 to R98, R31 to R99, U6 to U15, U5 to U16, U7 to U17

Commit message: add footprint
Parts:
- J22: footprint (none) -> IVS_FOOTPRINTS:HT - 3.96mm - 3pin
Changed lines of the file:
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@@
       (effects (font (size 1.27 1.27)) (justify left) hide)
     )
-    (property "Footprint" "" (id 2) (at 205.74 113.03 0)
+    (property "Footprint" "IVS_FOOTPRINTS:HT - 3.96mm - 3pin" (id 2) (at 205.74 113.03 0)
       (effects (font (size 1.27 1.27)) hide)
     )

Commit message: add all footprint
Parts:
- renumbered J22 to J11
Changed lines of the file:
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@@
   (symbol (lib_id "power:GND") (at 115.57 53.975 0) (unit 1)
     (in_bom yes) (on_board yes)
-    (property "Reference" "#PWR0152" (id 0) (at 115.57 60.325 0)
+    (property "Reference" "#PWR0156" (id 0) (at 115.57 60.325 0)
       (effects (font (size 1.27 1.27)) hide)
     )
@@
   (symbol (lib_id "power:GND") (at 77.47 97.79 0) (unit 1)
     (in_bom yes) (on_board yes)
-    (property "Reference" "#PWR0148" (id 0) (at 77.47 104.14 0)
+    (property "Reference" "#PWR0152" (id 0) (at 77.47 104.14 0)
       (effects (font (size 1.27 1.27)) hide)
     )
@@
   (symbol (lib_id "power:GND") (at 92.71 97.155 0) (unit 1)
     (in_bom yes) (on_board yes)
-    (property "Reference" "#PWR0150" (id 0) (at 92.71 103.505 0)
+    (property "Reference" "#PWR0154" (id 0) (at 92.71 103.505 0)
       (effects (font (size 1.27 1.27)) hide)
     )
@@
   (symbol (lib_id "power:VCC") (at 26.67 66.04 0) (unit 1)
     (in_bom yes) (on_board yes) (fields_autoplaced)
-    (property "Reference" "#PWR0145" (id 0) (at 26.67 69.85 0)
+    (property "Reference" "#PWR0149" (id 0) (at 26.67 69.85 0)
       (effects (font (size 1.27 1.27)) hide)
     )
@@
   (symbol (lib_id "power:GND") (at 63.5 97.79 0) (unit 1)
     (in_bom yes) (on_board yes)
-    (property "Reference" "#PWR0147" (id 0) (at 63.5 104.14 0)
+    (property "Reference" "#PWR0151" (id 0) (at 63.5 104.14 0)
       (effects (font (size 1.27 1.27)) hide)
     )
@@
   (symbol (lib_id "power:GND") (at 92.075 53.975 0) (unit 1)
     (in_bom yes) (on_board yes) (fields_autoplaced)
-    (property "Reference" "#PWR0149" (id 0) (at 92.075 60.325 0)
+    (property "Reference" "#PWR0153" (id 0) (at 92.075 60.325 0)
       (effects (font (size 1.27 1.27)) hide)
     )
@@
   (symbol (lib_id "power:GND") (at 145.415 75.565 0) (unit 1)
     (in_bom yes) (on_board yes)
-    (property "Reference" "#PWR0153" (id 0) (at 145.415 81.915 0)
+    (property "Reference" "#PWR0157" (id 0) (at 145.415 81.915 0)
       (effects (font (size 1.27 1.27)) hide)
     )
@@
   (symbol (lib_id "power:VCC") (at 198.12 104.14 0) (unit 1)
     (in_bom yes) (on_board yes) (fields_autoplaced)
-    (property "Reference" "#PWR0156" (id 0) (at 198.12 107.95 0)
+    (property "Reference" "#PWR0160" (id 0) (at 198.12 107.95 0)
       (effects (font (size 1.27 1.27)) hide)
     )
@@
   (symbol (lib_id "power:GND") (at 198.12 118.11 0) (unit 1)
     (in_bom yes) (on_board yes)
-    (property "Reference" "#PWR0157" (id 0) (at 198.12 124.46 0)
+    (property "Reference" "#PWR0161" (id 0) (at 198.12 124.46 0)
       (effects (font (size 1.27 1.27)) hide)
     )
@@
   (symbol (lib_id "power:GND") (at 26.67 102.235 0) (unit 1)
     (in_bom yes) (on_board yes) (fields_autoplaced)
-    (property "Reference" "#PWR0146" (id 0) (at 26.67 108.585 0)
+    (property "Reference" "#PWR0150" (id 0) (at 26.67 108.585 0)
       (effects (font (size 1.27 1.27)) hide)
     )
@@
   (symbol (lib_id "power:GND") (at 152.4 75.565 0) (unit 1)
     (in_bom yes) (on_board yes)
-    (property "Reference" "#PWR0154" (id 0) (at 152.4 81.915 0)
+    (property "Reference" "#PWR0158" (id 0) (at 152.4 81.915 0)
       (effects (font (size 1.27 1.27)) hide)
     )
@@
   (symbol (lib_id "power:GND") (at 160.655 107.315 0) (unit 1)
     (in_bom yes) (on_board yes)
-    (property "Reference" "#PWR0155" (id 0) (at 160.655 113.665 0)
+    (property "Reference" "#PWR0159" (id 0) (at 160.655 113.665 0)
       (effects (font (size 1.27 1.27)) hide)
     )
@@
   (symbol (lib_id "power:GND") (at 111.125 97.79 0) (unit 1)
     (in_bom yes) (on_board yes)
-    (property "Reference" "#PWR0151" (id 0) (at 111.125 104.14 0)
+    (property "Reference" "#PWR0155" (id 0) (at 111.125 104.14 0)
       (effects (font (size 1.27 1.27)) hide)
     )
@@
   (symbol (lib_id "Connector:Screw_Terminal_01x03") (at 205.74 113.03 0) (unit 1)
     (in_bom yes) (on_board yes) (fields_autoplaced)
-    (property "Reference" "J22" (id 0) (at 208.915 113.0299 0)
-      (effects (font (size 1.27 1.27)) (justify left))
-    )
+    (property "Reference" "J11" (id 0) (at 208.915 113.0299 0)
+      (effects (font (size 1.27 1.27)) (justify left))
+    )

Commit message: add shematics MVA
Connections:
- net GND: now also J11.1 (Pin_1); no longer J11.3 (Pin_3)
- net VCC: now also J11.3 (Pin_3); no longer J11.1 (Pin_1)
Changed lines of the file:
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@@
     )
   )
-  (symbol (lib_id "Connector:Screw_Terminal_01x03") (at 205.74 113.03 0) (unit 1)
-    (in_bom yes) (on_board yes) (dnp no) (fields_autoplaced)
-    (property "Reference" "J11" (at 208.915 113.0299 0)
+  (symbol (lib_id "Connector:Screw_Terminal_01x03") (at 205.74 113.03 0) (mirror x) (unit 1)
+    (in_bom yes) (on_board yes) (dnp no)
+    (property "Reference" "J11" (at 208.915 113.0301 0)
       (effects (font (size 1.27 1.27)) (justify left))
     )
-    (property "Value" "Screw_Terminal" (at 208.28 114.2999 0)
+    (property "Value" "Screw_Terminal" (at 208.28 111.7601 0)
       (effects (font (size 1.27 1.27)) (justify left) hide)
     )
