File: Hardware/4-20mAConverter.kicad_sch (KiCad schematic)
At the start: 26 parts, among them J11 HT3.96mm-3P, Q17 NPN, U15 LM324, U16 LM317_TO-252, U17 TL431

Commit message: add lora, relay, opto, opamp block, led for 74595. Delete RT9193, connect boot0,1 to GND. Fix footprint crystal 8M, 74HC595, IDC pin
Parts:
- C32: footprint IVS_FOOTPRINTS:C0603 -> IVS_FOOTPRINTS:C_0603
- LE1: footprint IVS_FOOTPRINTS:LED0603 -> IVS_FOOTPRINTS:LED_0603
- LE2: footprint IVS_FOOTPRINTS:LED0805 -> IVS_FOOTPRINTS:LED_0603
- R100, R101, R102, R103, R104, R105, R106, R107, R108, R109, R95, R96, R97, R98, R99: footprint IVS_FOOTPRINTS:R0603 -> IVS_FOOTPRINTS:R_0603
- U16: footprint Package_TO_SOT_SMD:TO-252-2 -> IVS_FOOTPRINTS:TO-252-2
Changed lines of the file:
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@@
     (effects (font (size 1.27 1.27)) (justify right))
   )
-  (symbol (lib_id "power:GND") (at 115.57 53.975 0) (unit 1)
+  (symbol (lib_name "GND_7") (lib_id "power:GND") (at 115.57 53.975 0) (unit 1)
     (in_bom yes) (on_board yes) (dnp no)
     (property "Reference" "#PWR0156" (at 115.57 60.325 0)
@@
       (effects (font (size 1.27 1.27)))
     )
-    (property "Footprint" "IVS_FOOTPRINTS:R0603" (at 128.27 50.673 90)
+    (property "Footprint" "IVS_FOOTPRINTS:R_0603" (at 128.27 50.673 90)
       (effects (font (size 1.27 1.27)) hide)
     )
@@
       (effects (font (size 1.27 1.27)))
     )
-    (property "Footprint" "IVS_FOOTPRINTS:R0603" (at 168.91 63.373 90)
+    (property "Footprint" "IVS_FOOTPRINTS:R_0603" (at 168.91 63.373 90)
       (effects (font (size 1.27 1.27)) hide)
     )
@@
       (effects (font (size 1.27 1.27)))
     )
-    (property "Footprint" "IVS_FOOTPRINTS:R0603" (at 86.36 70.612 90)
+    (property "Footprint" "IVS_FOOTPRINTS:R_0603" (at 86.36 70.612 90)
       (effects (font (size 1.27 1.27)) hide)
     )
@@
       (effects (font (size 1.27 1.27)) (justify left))
     )
-    (property "Footprint" "IVS_FOOTPRINTS:R0603" (at 150.622 67.945 90)
+    (property "Footprint" "IVS_FOOTPRINTS:R_0603" (at 150.622 67.945 90)
       (effects (font (size 1.27 1.27)) hide)
     )
@@
       (effects (font (size 1.27 1.27)) (justify left))
     )
-    (property "Footprint" "IVS_FOOTPRINTS:R0603" (at 90.297 36.195 90)
+    (property "Footprint" "IVS_FOOTPRINTS:R_0603" (at 90.297 36.195 90)
       (effects (font (size 1.27 1.27)) hide)
     )
@@
     )
   )
-  (symbol (lib_id "power:GND") (at 92.71 97.155 0) (unit 1)
+  (symbol (lib_name "GND_6") (lib_id "power:GND") (at 92.71 97.155 0) (unit 1)
     (in_bom yes) (on_board yes) (dnp no)
     (property "Reference" "#PWR0154" (at 92.71 103.505 0)
@@
       (effects (font (size 1.27 1.27)))
     )
-    (property "Footprint" "Package_TO_SOT_SMD:TO-252-2" (at 53.34 66.04 0)
+    (property "Footprint" "IVS_FOOTPRINTS:TO-252-2" (at 53.34 66.04 0)
       (effects (font (size 1.27 1.27) italic) hide)
     )
@@
       (effects (font (size 1.27 1.27)) (justify left))
     )
-    (property "Footprint" "IVS_FOOTPRINTS:C0603" (at 39.0652 93.345 0)
+    (property "Footprint" "IVS_FOOTPRINTS:C_0603" (at 39.0652 93.345 0)
       (effects (font (size 1.27 1.27)) hide)
     )
@@
     )
   )
-  (symbol (lib_id "power:GND") (at 63.5 97.79 0) (unit 1)
+  (symbol (lib_name "GND_5") (lib_id "power:GND") (at 63.5 97.79 0) (unit 1)
     (in_bom yes) (on_board yes) (dnp no)
     (property "Reference" "#PWR0151" (at 63.5 104.14 0)
@@
       (effects (font (size 1.27 1.27)) (justify right))
     )
-    (property "Footprint" "IVS_FOOTPRINTS:R0603" (at 163.957 99.695 90)
+    (property "Footprint" "IVS_FOOTPRINTS:R_0603" (at 163.957 99.695 90)
       (effects (font (size 1.27 1.27)) hide)
     )
@@
     )
   )
-  (symbol (lib_id "power:GND") (at 92.075 53.975 0) (unit 1)
+  (symbol (lib_name "GND_4") (lib_id "power:GND") (at 92.075 53.975 0) (unit 1)
     (in_bom yes) (on_board yes) (dnp no) (fields_autoplaced)
     (property "Reference" "#PWR0153" (at 92.075 60.325 0)
@@
     )
   )
-  (symbol (lib_id "IVS_SYMBOLS:Led") (at 190.5 113.03 180) (unit 1)
+  (symbol (lib_name "Led_1") (lib_id "IVS_SYMBOLS:Led") (at 190.5 113.03 180) (unit 1)
     (in_bom yes) (on_board yes) (dnp no) (fields_autoplaced)
     (property "Reference" "LE2" (at 190.8175 105.41 0)
@@
       (effects (font (size 1.27 1.27)))
     )
-    (property "Footprint" "IVS_FOOTPRINTS:LED0805" (at 189.738 112.776 0)
+    (property "Footprint" "IVS_FOOTPRINTS:LED_0603" (at 189.738 112.776 0)
       (effects (font (size 1.27 1.27)) hide)
     )
@@
     )
   )
-  (symbol (lib_id "power:VCC") (at 198.12 104.14 0) (unit 1)
+  (symbol (lib_name "VCC_1") (lib_id "power:VCC") (at 198.12 104.14 0) (unit 1)
     (in_bom yes) (on_board yes) (dnp no) (fields_autoplaced)
     (property "Reference" "#PWR0160" (at 198.12 107.95 0)
@@
       (effects (font (size 1.27 1.27)) (justify right))
     )
-    (property "Footprint" "IVS_FOOTPRINTS:R0603" (at 170.815 111.252 90)
+    (property "Footprint" "IVS_FOOTPRINTS:R_0603" (at 170.815 111.252 90)
       (effects (font (size 1.27 1.27)) hide)
     )
@@
       (effects (font (size 1.27 1.27)) (justify left))
     )
-    (property "Footprint" "IVS_FOOTPRINTS:R0603" (at 61.722 91.44 90)
+    (property "Footprint" "IVS_FOOTPRINTS:R_0603" (at 61.722 91.44 90)
       (effects (font (size 1.27 1.27)) hide)
     )
@@
     )
   )
-  (symbol (lib_id "power:GND") (at 198.12 118.11 0) (unit 1)
+  (symbol (lib_name "GND_9") (lib_id "power:GND") (at 198.12 118.11 0) (unit 1)
     (in_bom yes) (on_board yes) (dnp no)
     (property "Reference" "#PWR0161" (at 198.12 124.46 0)
@@
     )
   )
-  (symbol (lib_id "power:GND") (at 26.67 102.235 0) (unit 1)
+  (symbol (lib_name "GND_8") (lib_id "power:GND") (at 26.67 102.235 0) (unit 1)
     (in_bom yes) (on_board yes) (dnp no) (fields_autoplaced)
     (property "Reference" "#PWR0150" (at 26.67 108.585 0)
@@
       (effects (font (size 1.27 1.27)) (justify left))
     )
-    (property "Footprint" "IVS_FOOTPRINTS:R0603" (at 75.692 76.2 90)
+    (property "Footprint" "IVS_FOOTPRINTS:R_0603" (at 75.692 76.2 90)
       (effects (font (size 1.27 1.27)) hide)
     )
@@
       (effects (font (size 1.27 1.27)) (justify left))
     )
-    (property "Footprint" "IVS_FOOTPRINTS:R0603" (at 176.022 78.74 90)
+    (property "Footprint" "IVS_FOOTPRINTS:R_0603" (at 176.022 78.74 90)
       (effects (font (size 1.27 1.27)) hide)
     )
@@
       (effects (font (size 1.27 1.27)) (justify right))
     )
-    (property "Footprint" "IVS_FOOTPRINTS:LED0603" (at 77.724 88.138 0)
+    (property "Footprint" "IVS_FOOTPRINTS:LED_0603" (at 77.724 88.138 0)
       (effects (font (size 1.27 1.27)) hide)
     )
@@
       (effects (font (size 1.27 1.27)) (justify left))
     )
-    (property "Footprint" "IVS_FOOTPRINTS:R0603" (at 158.877 99.695 90)
+    (property "Footprint" "IVS_FOOTPRINTS:R_0603" (at 158.877 99.695 90)
       (effects (font (size 1.27 1.27)) hide)
     )
@@
     )
   )
-  (symbol (lib_id "power:GND") (at 152.4 75.565 0) (unit 1)
+  (symbol (lib_name "GND_3") (lib_id "power:GND") (at 152.4 75.565 0) (unit 1)
     (in_bom yes) (on_board yes) (dnp no)
     (property "Reference" "#PWR0158" (at 152.4 81.915 0)
@@
       (effects (font (size 1.27 1.27)) (justify left))
     )
-    (property "Footprint" "IVS_FOOTPRINTS:R0603" (at 61.722 80.01 90)
+    (property "Footprint" "IVS_FOOTPRINTS:R_0603" (at 61.722 80.01 90)
       (effects (font (size 1.27 1.27)) hide)
     )
@@
     )
   )
-  (symbol (lib_id "power:GND") (at 160.655 107.315 0) (unit 1)
+  (symbol (lib_name "GND_2") (lib_id "power:GND") (at 160.655 107.315 0) (unit 1)
     (in_bom yes) (on_board yes) (dnp no)
     (property "Reference" "#PWR0159" (at 160.655 113.665 0)
@@
     )
   )
-  (symbol (lib_id "power:GND") (at 111.125 97.79 0) (unit 1)
+  (symbol (lib_name "GND_1") (lib_id "power:GND") (at 111.125 97.79 0) (unit 1)
     (in_bom yes) (on_board yes) (dnp no)
     (property "Reference" "#PWR0155" (at 111.125 104.14 0)
@@
       (effects (font (size 1.27 1.27)) (justify right))
     )
-    (property "Footprint" "IVS_FOOTPRINTS:R0603" (at 176.022 94.615 90)
+    (property "Footprint" "IVS_FOOTPRINTS:R_0603" (at 176.022 94.615 90)
       (effects (font (size 1.27 1.27)) hide)
     )
@@
       (effects (font (size 1.27 1.27)))
     )
-    (property "Footprint" "IVS_FOOTPRINTS:R0603" (at 100.33 70.612 90)
+    (property "Footprint" "IVS_FOOTPRINTS:R_0603" (at 100.33 70.612 90)
       (effects (font (size 1.27 1.27)) hide)
     )
@@
       (effects (font (size 1.27 1.27)) (justify left))
     )
-    (property "Footprint" "IVS_FOOTPRINTS:R0603" (at 141.097 62.865 90)
-      (effects (font (size 1.27 1.27)) hide)
-    )
+    (property "Footprint" "IVS_FOOTPRINTS:R_0603" (at 141.097 62.865 90)
+      (effects (font (size 1.27 1.27)) hide)
+    )
