File: Hardware/1_TL084IPT.kicad_sch (KiCad schematic)
At the start: 27 parts, among them Q1 SI_2300, Q2 SI_2300, Q3 SI_2300, Q4 SI_2300, U11 TL084

Commit message: add all footprint
Parts:
- gave numbers to parts that had none: 1
Changed lines of the file:
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@@
   (symbol (lib_id "power:GND") (at 93.98 191.77 0) (unit 1)
     (in_bom yes) (on_board yes) (fields_autoplaced)
-    (property "Reference" "#PWR082" (id 0) (at 93.98 198.12 0)
+    (property "Reference" "#PWR086" (id 0) (at 93.98 198.12 0)
       (effects (font (size 1.27 1.27)) hide)
     )
@@
   (symbol (lib_id "power:+24V") (at 72.39 109.22 0) (unit 1)
     (in_bom yes) (on_board yes) (fields_autoplaced)
-    (property "Reference" "#PWR073" (id 0) (at 72.39 113.03 0)
+    (property "Reference" "#PWR077" (id 0) (at 72.39 113.03 0)
       (effects (font (size 1.27 1.27)) hide)
     )
@@
   (symbol (lib_id "power:+3V3") (at 119.38 77.47 0) (unit 1)
     (in_bom yes) (on_board yes) (fields_autoplaced)
-    (property "Reference" "#PWR085" (id 0) (at 119.38 81.28 0)
+    (property "Reference" "#PWR089" (id 0) (at 119.38 81.28 0)
       (effects (font (size 1.27 1.27)) hide)
     )
@@
   (symbol (lib_id "power:+24V") (at 72.39 20.32 0) (unit 1)
     (in_bom yes) (on_board yes) (fields_autoplaced)
-    (property "Reference" "#PWR069" (id 0) (at 72.39 24.13 0)
+    (property "Reference" "#PWR073" (id 0) (at 72.39 24.13 0)
       (effects (font (size 1.27 1.27)) hide)
     )
@@
   (symbol (lib_id "power:GND") (at 93.98 146.05 0) (unit 1)
     (in_bom yes) (on_board yes) (fields_autoplaced)
-    (property "Reference" "#PWR081" (id 0) (at 93.98 152.4 0)
+    (property "Reference" "#PWR085" (id 0) (at 93.98 152.4 0)
       (effects (font (size 1.27 1.27)) hide)
     )
@@
   (symbol (lib_id "Connector:Screw_Terminal_01x08") (at 28.575 103.505 0) (mirror y) (unit 1)
     (in_bom yes) (on_board yes) (fields_autoplaced)
-    (property "Reference" "J?" (id 0) (at 28.575 89.535 0))
+    (property "Reference" "J7" (id 0) (at 28.575 89.535 0))
     (property "Value" "Screw_Terminal_01x08" (id 1) (at 28.575 92.075 0))
     (property "Footprint" "IVS_FOOTPRINTS:HT-3.96mm" (id 2) (at 28.575 103.505 0)
@@
   (symbol (lib_id "power:GND") (at 86.36 33.02 0) (unit 1)
     (in_bom yes) (on_board yes)
-    (property "Reference" "#PWR078" (id 0) (at 86.36 39.37 0)
+    (property "Reference" "#PWR082" (id 0) (at 86.36 39.37 0)
       (effects (font (size 1.27 1.27)) hide)
     )
@@
   (symbol (lib_id "power:+24V") (at 72.39 64.77 0) (unit 1)
     (in_bom yes) (on_board yes) (fields_autoplaced)
-    (property "Reference" "#PWR071" (id 0) (at 72.39 68.58 0)
+    (property "Reference" "#PWR075" (id 0) (at 72.39 68.58 0)
       (effects (font (size 1.27 1.27)) hide)
     )
@@
   (symbol (lib_id "power:GND") (at 93.98 57.15 0) (unit 1)
     (in_bom yes) (on_board yes) (fields_autoplaced)
-    (property "Reference" "#PWR079" (id 0) (at 93.98 63.5 0)
+    (property "Reference" "#PWR083" (id 0) (at 93.98 63.5 0)
       (effects (font (size 1.27 1.27)) hide)
     )
@@
   (symbol (lib_id "power:GND") (at 72.39 186.69 0) (unit 1)
     (in_bom yes) (on_board yes) (fields_autoplaced)
-    (property "Reference" "#PWR076" (id 0) (at 72.39 193.04 0)
+    (property "Reference" "#PWR080" (id 0) (at 72.39 193.04 0)
       (effects (font (size 1.27 1.27)) hide)
     )
@@
   (symbol (lib_id "power:+3V3") (at 86.36 25.4 0) (unit 1)
     (in_bom yes) (on_board yes) (fields_autoplaced)
-    (property "Reference" "#PWR077" (id 0) (at 86.36 29.21 0)
+    (property "Reference" "#PWR081" (id 0) (at 86.36 29.21 0)
       (effects (font (size 1.27 1.27)) hide)
     )
@@
   (symbol (lib_id "power:GND") (at 72.39 142.24 0) (unit 1)
     (in_bom yes) (on_board yes) (fields_autoplaced)
-    (property "Reference" "#PWR074" (id 0) (at 72.39 148.59 0)
+    (property "Reference" "#PWR078" (id 0) (at 72.39 148.59 0)
       (effects (font (size 1.27 1.27)) hide)
     )
@@
   (symbol (lib_id "power:+24V") (at 72.39 153.67 0) (unit 1)
     (in_bom yes) (on_board yes)
-    (property "Reference" "#PWR075" (id 0) (at 72.39 157.48 0)
+    (property "Reference" "#PWR079" (id 0) (at 72.39 157.48 0)
       (effects (font (size 1.27 1.27)) hide)
     )
@@
   (symbol (lib_id "power:+3V3") (at 119.38 120.65 0) (unit 1)
     (in_bom yes) (on_board yes) (fields_autoplaced)
-    (property "Reference" "#PWR086" (id 0) (at 119.38 124.46 0)
+    (property "Reference" "#PWR090" (id 0) (at 119.38 124.46 0)
       (effects (font (size 1.27 1.27)) hide)
     )
@@
   (symbol (lib_id "power:GND") (at 107.95 25.4 0) (unit 1)
     (in_bom yes) (on_board yes) (fields_autoplaced)
-    (property "Reference" "#PWR083" (id 0) (at 107.95 31.75 0)
+    (property "Reference" "#PWR087" (id 0) (at 107.95 31.75 0)
       (effects (font (size 1.27 1.27)) hide)
     )
@@
   (symbol (lib_id "power:+3V3") (at 119.38 166.37 0) (unit 1)
     (in_bom yes) (on_board yes) (fields_autoplaced)
-    (property "Reference" "#PWR087" (id 0) (at 119.38 170.18 0)
+    (property "Reference" "#PWR091" (id 0) (at 119.38 170.18 0)
       (effects (font (size 1.27 1.27)) hide)
     )
@@
   (symbol (lib_id "power:GND") (at 72.39 97.79 0) (unit 1)
     (in_bom yes) (on_board yes) (fields_autoplaced)
-    (property "Reference" "#PWR072" (id 0) (at 72.39 104.14 0)
+    (property "Reference" "#PWR076" (id 0) (at 72.39 104.14 0)
       (effects (font (size 1.27 1.27)) hide)
     )
@@
   (symbol (lib_id "power:GND") (at 72.39 52.07 0) (unit 1)
     (in_bom yes) (on_board yes) (fields_autoplaced)
-    (property "Reference" "#PWR070" (id 0) (at 72.39 58.42 0)
+    (property "Reference" "#PWR074" (id 0) (at 72.39 58.42 0)
       (effects (font (size 1.27 1.27)) hide)
     )
@@
   (symbol (lib_id "power:GND") (at 93.98 102.87 0) (unit 1)
     (in_bom yes) (on_board yes) (fields_autoplaced)
-    (property "Reference" "#PWR080" (id 0) (at 93.98 109.22 0)
+    (property "Reference" "#PWR084" (id 0) (at 93.98 109.22 0)
       (effects (font (size 1.27 1.27)) hide)
     )
@@
   (symbol (lib_id "power:+3V3") (at 119.38 31.75 0) (unit 1)
     (in_bom yes) (on_board yes) (fields_autoplaced)
-    (property "Reference" "#PWR084" (id 0) (at 119.38 35.56 0)
-      (effects (font (size 1.27 1.27)) hide)
-    )
+    (property "Reference" "#PWR088" (id 0) (at 119.38 35.56 0)
+      (effects (font (size 1.27 1.27)) hide)
+    )

Commit message: add shematics MVA
Parts:
- removed R39, R40, R41, R42: 1k, IVS_FOOTPRINTS:R0603, symbol Device:R

Commit message: layout PCB part 1
Parts:
- removed Q1, Q2, Q3, Q4: SI_2300, IVS_FOOTPRINTS:SOT23-3, symbol Device:Q_NMOS_DGS
- added Q1, Q2, Q20, Q3: N_Mosfet, IVS_FOOTPRINTS:SOT23-3, symbol IVS_SYMBOLS:N_Mosfet
Connections:
- net VAN1-: now also J7.8 (Pin_8), Q20.3 (D); no longer J7.2 (Pin_2)
- net VAN1_input: now also Q20.1 (G)
- net VAN2-: now also J7.6 (Pin_6), Q1.3 (D); no longer J7.4 (Pin_4)
- net VAN2_input: now also Q1.1 (G)
- net VAN3-: now also J7.4 (Pin_4), Q2.3 (D); no longer J7.6 (Pin_6)
- net VAN3_input: now also Q2.1 (G)
- net VAN4-: now also J7.2 (Pin_2), Q3.3 (D); no longer J7.8 (Pin_8)
- net VAN4_input: now also Q3.1 (G)
- net at R38.1, U11.12 (+): now also Q3.2 (S)
- net at R35.1, U11.3 (+): now also Q20.2 (S)
- net at R37.1, U11.10 (+): now also Q2.2 (S)
- net at R36.1, U11.5 (+): now also Q1.2 (S)
