File: Hardware/2_TL084IPT.kicad_sch (KiCad schematic)
At the start: 27 parts, among them Q5 SI_2300, Q6 SI_2300, Q7 SI_2300, Q8 SI_2300, U12 TL084

Commit message: add all footprint
Parts:
- gave numbers to parts that had none: 1
Changed lines of the file:
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@@
   (symbol (lib_id "Connector:Screw_Terminal_01x08") (at 21.59 99.06 0) (mirror y) (unit 1)
     (in_bom yes) (on_board yes) (fields_autoplaced)
-    (property "Reference" "J?" (id 0) (at 21.59 85.09 0))
+    (property "Reference" "J8" (id 0) (at 21.59 85.09 0))
     (property "Value" "Screw_Terminal_01x08" (id 1) (at 21.59 87.63 0))
     (property "Footprint" "IVS_FOOTPRINTS:HT-3.96mm" (id 2) (at 21.59 99.06 0)
@@
   (symbol (lib_id "power:+24V") (at 67.31 106.68 0) (unit 1)
     (in_bom yes) (on_board yes) (fields_autoplaced)
-    (property "Reference" "#PWR092" (id 0) (at 67.31 110.49 0)
+    (property "Reference" "#PWR096" (id 0) (at 67.31 110.49 0)
       (effects (font (size 1.27 1.27)) hide)
     )
@@
   (symbol (lib_id "power:+3V3") (at 114.3 163.83 0) (unit 1)
     (in_bom yes) (on_board yes) (fields_autoplaced)
-    (property "Reference" "#PWR0106" (id 0) (at 114.3 167.64 0)
+    (property "Reference" "#PWR0110" (id 0) (at 114.3 167.64 0)
       (effects (font (size 1.27 1.27)) hide)
     )
@@
   (symbol (lib_id "power:+3V3") (at 114.3 74.93 0) (unit 1)
     (in_bom yes) (on_board yes) (fields_autoplaced)
-    (property "Reference" "#PWR0104" (id 0) (at 114.3 78.74 0)
+    (property "Reference" "#PWR0108" (id 0) (at 114.3 78.74 0)
       (effects (font (size 1.27 1.27)) hide)
     )
@@
   (symbol (lib_id "power:+24V") (at 67.31 17.78 0) (unit 1)
     (in_bom yes) (on_board yes) (fields_autoplaced)
-    (property "Reference" "#PWR088" (id 0) (at 67.31 21.59 0)
+    (property "Reference" "#PWR092" (id 0) (at 67.31 21.59 0)
       (effects (font (size 1.27 1.27)) hide)
     )
@@
   (symbol (lib_id "power:+24V") (at 67.31 151.13 0) (unit 1)
     (in_bom yes) (on_board yes) (fields_autoplaced)
-    (property "Reference" "#PWR094" (id 0) (at 67.31 154.94 0)
+    (property "Reference" "#PWR098" (id 0) (at 67.31 154.94 0)
       (effects (font (size 1.27 1.27)) hide)
     )
@@
   (symbol (lib_id "power:+3V3") (at 81.28 22.86 0) (unit 1)
     (in_bom yes) (on_board yes) (fields_autoplaced)
-    (property "Reference" "#PWR096" (id 0) (at 81.28 26.67 0)
+    (property "Reference" "#PWR0100" (id 0) (at 81.28 26.67 0)
       (effects (font (size 1.27 1.27)) hide)
     )
@@
   (symbol (lib_id "power:+24V") (at 67.31 62.23 0) (unit 1)
     (in_bom yes) (on_board yes) (fields_autoplaced)
-    (property "Reference" "#PWR090" (id 0) (at 67.31 66.04 0)
+    (property "Reference" "#PWR094" (id 0) (at 67.31 66.04 0)
       (effects (font (size 1.27 1.27)) hide)
     )
@@
   (symbol (lib_id "power:GND") (at 102.87 22.86 0) (unit 1)
     (in_bom yes) (on_board yes) (fields_autoplaced)
-    (property "Reference" "#PWR0102" (id 0) (at 102.87 29.21 0)
+    (property "Reference" "#PWR0106" (id 0) (at 102.87 29.21 0)
       (effects (font (size 1.27 1.27)) hide)
     )
@@
   (symbol (lib_id "power:GND") (at 67.31 139.7 0) (unit 1)
     (in_bom yes) (on_board yes) (fields_autoplaced)
-    (property "Reference" "#PWR093" (id 0) (at 67.31 146.05 0)
+    (property "Reference" "#PWR097" (id 0) (at 67.31 146.05 0)
       (effects (font (size 1.27 1.27)) hide)
     )
@@
   (symbol (lib_id "power:GND") (at 67.31 95.25 0) (unit 1)
     (in_bom yes) (on_board yes) (fields_autoplaced)
-    (property "Reference" "#PWR091" (id 0) (at 67.31 101.6 0)
+    (property "Reference" "#PWR095" (id 0) (at 67.31 101.6 0)
       (effects (font (size 1.27 1.27)) hide)
     )
@@
   (symbol (lib_id "power:GND") (at 88.9 189.23 0) (unit 1)
     (in_bom yes) (on_board yes) (fields_autoplaced)
-    (property "Reference" "#PWR0101" (id 0) (at 88.9 195.58 0)
+    (property "Reference" "#PWR0105" (id 0) (at 88.9 195.58 0)
       (effects (font (size 1.27 1.27)) hide)
     )
@@
   (symbol (lib_id "power:GND") (at 81.28 30.48 0) (unit 1)
     (in_bom yes) (on_board yes)
-    (property "Reference" "#PWR097" (id 0) (at 81.28 36.83 0)
+    (property "Reference" "#PWR0101" (id 0) (at 81.28 36.83 0)
       (effects (font (size 1.27 1.27)) hide)
     )
@@
   (symbol (lib_id "power:GND") (at 67.31 49.53 0) (unit 1)
     (in_bom yes) (on_board yes) (fields_autoplaced)
-    (property "Reference" "#PWR089" (id 0) (at 67.31 55.88 0)
+    (property "Reference" "#PWR093" (id 0) (at 67.31 55.88 0)
       (effects (font (size 1.27 1.27)) hide)
     )
@@
   (symbol (lib_id "power:+3V3") (at 114.3 118.11 0) (unit 1)
     (in_bom yes) (on_board yes) (fields_autoplaced)
-    (property "Reference" "#PWR0105" (id 0) (at 114.3 121.92 0)
+    (property "Reference" "#PWR0109" (id 0) (at 114.3 121.92 0)
       (effects (font (size 1.27 1.27)) hide)
     )
@@
   (symbol (lib_id "power:+3V3") (at 114.3 29.21 0) (unit 1)
     (in_bom yes) (on_board yes) (fields_autoplaced)
-    (property "Reference" "#PWR0103" (id 0) (at 114.3 33.02 0)
+    (property "Reference" "#PWR0107" (id 0) (at 114.3 33.02 0)
       (effects (font (size 1.27 1.27)) hide)
     )
@@
   (symbol (lib_id "power:GND") (at 88.9 143.51 0) (unit 1)
     (in_bom yes) (on_board yes) (fields_autoplaced)
-    (property "Reference" "#PWR0100" (id 0) (at 88.9 149.86 0)
+    (property "Reference" "#PWR0104" (id 0) (at 88.9 149.86 0)
       (effects (font (size 1.27 1.27)) hide)
     )
@@
   (symbol (lib_id "power:GND") (at 88.9 54.61 0) (unit 1)
     (in_bom yes) (on_board yes) (fields_autoplaced)
-    (property "Reference" "#PWR098" (id 0) (at 88.9 60.96 0)
+    (property "Reference" "#PWR0102" (id 0) (at 88.9 60.96 0)
       (effects (font (size 1.27 1.27)) hide)
     )
@@
   (symbol (lib_id "power:GND") (at 88.9 100.33 0) (unit 1)
     (in_bom yes) (on_board yes) (fields_autoplaced)
-    (property "Reference" "#PWR099" (id 0) (at 88.9 106.68 0)
+    (property "Reference" "#PWR0103" (id 0) (at 88.9 106.68 0)
       (effects (font (size 1.27 1.27)) hide)
     )
@@
   (symbol (lib_id "power:GND") (at 67.31 184.15 0) (unit 1)
     (in_bom yes) (on_board yes) (fields_autoplaced)
-    (property "Reference" "#PWR095" (id 0) (at 67.31 190.5 0)
-      (effects (font (size 1.27 1.27)) hide)
-    )
+    (property "Reference" "#PWR099" (id 0) (at 67.31 190.5 0)
+      (effects (font (size 1.27 1.27)) hide)
+    )

Commit message: add shematics MVA
Parts:
- removed R55, R56, R57, R58: 1k, IVS_FOOTPRINTS:R0603, symbol Device:R
Changed lines of the file:
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@@
-    (stroke (width 0) (type default))
-  )
-  (wire (pts (xy 88.9 100.33) (xy 88.9 99.06))
     (stroke (width 0) (type default))
   )
@@
     (stroke (width 0) (type default))
   )
-  (wire (pts (xy 88.9 134.62) (xy 88.9 133.35))
-    (stroke (width 0) (type default))
-  )
   (wire (pts (xy 55.88 111.76) (xy 55.88 107.95))
     (stroke (width 0) (type default))
@@
     (stroke (width 0) (type default))
   )
-  (wire (pts (xy 88.9 45.72) (xy 88.9 44.45))
-    (stroke (width 0) (type default))
-  )
   (wire (pts (xy 67.31 62.23) (xy 67.31 63.5))
     (stroke (width 0) (type default))
@@
     (stroke (width 0) (type default))
   )
-  (wire (pts (xy 88.9 143.51) (xy 88.9 142.24))
-    (stroke (width 0) (type default))
-  )
   (wire (pts (xy 67.31 137.16) (xy 67.31 139.7))
     (stroke (width 0) (type default))
@@
     (stroke (width 0) (type default))
   )
-  (wire (pts (xy 88.9 54.61) (xy 88.9 53.34))
-    (stroke (width 0) (type default))
-  )
   (wire (pts (xy 67.31 116.84) (xy 67.31 118.11))
     (stroke (width 0) (type default))
@@
     (stroke (width 0) (type default))
   )
-  (wire (pts (xy 88.9 180.34) (xy 88.9 179.07))
-    (stroke (width 0) (type default))
-  )
   (wire (pts (xy 49.53 67.31) (xy 54.61 67.31))
     (stroke (width 0) (type default))
@@
     (stroke (width 0) (type default))
   )
-  (wire (pts (xy 88.9 189.23) (xy 88.9 187.96))
-    (stroke (width 0) (type default))
-  )
   (wire (pts (xy 50.8 158.75) (xy 55.88 158.75))
     (stroke (width 0) (type default))
@@
   )
   (wire (pts (xy 55.88 33.02) (xy 59.69 33.02))
-    (stroke (width 0) (type default))
-  )
-  (wire (pts (xy 88.9 91.44) (xy 88.9 90.17))
     (stroke (width 0) (type default))
   )
@@
     )
   )
-  (symbol (lib_id "Device:R") (at 88.9 95.25 0) (unit 1)
-    (in_bom yes) (on_board yes) (dnp no)
-    (property "Reference" "R56" (at 90.17 93.98 0)
-      (effects (font (size 1.27 1.27)) (justify left))
-    )
-    (property "Value" "1k" (at 90.17 96.52 0)
-      (effects (font (size 1.27 1.27)) (justify left))
-    )
-    (property "Footprint" "IVS_FOOTPRINTS:R0603" (at 87.122 95.25 90)
-      (effects (font (size 1.27 1.27)) hide)
-    )
-    (property "Datasheet" "~" (at 88.9 95.25 0)
-      (effects (font (size 1.27 1.27)) hide)
-    )
-    (pin "1")
-    (pin "2")
-    (instances
-      (project "dongtam"
-        (path "/6833aec4-3d1d-4261-9b3e-f0452b565dd3/992d1183-82f3-4ab3-a77f-7ab8cf195fcd/e4ad1a02-817a-4cce-9ee6-266c75a94756/9d30bcf3-6fd4-4ecd-bcd6-7dfab3ad93fc"
-          (reference "R56") (unit 1)
-        )
-      )
-    )
-  )
   (symbol (lib_id "power:+3V3") (at 81.28 22.86 0) (unit 1)
     (in_bom yes) (on_board yes) (dnp no) (fields_autoplaced)
@@
     )
   )
-  (symbol (lib_id "Device:R") (at 88.9 138.43 0) (unit 1)
-    (in_bom yes) (on_board yes) (dnp no)
-    (property "Reference" "R57" (at 90.17 137.16 0)
-      (effects (font (size 1.27 1.27)) (justify left))
-    )
-    (property "Value" "1k" (at 90.17 139.7 0)
-      (effects (font (size 1.27 1.27)) (justify left))
-    )
-    (property "Footprint" "IVS_FOOTPRINTS:R0603" (at 87.122 138.43 90)
-      (effects (font (size 1.27 1.27)) hide)
-    )
-    (property "Datasheet" "~" (at 88.9 138.43 0)
-      (effects (font (size 1.27 1.27)) hide)
-    )
-    (pin "1")
-    (pin "2")
-    (instances
-      (project "dongtam"
-        (path "/6833aec4-3d1d-4261-9b3e-f0452b565dd3/992d1183-82f3-4ab3-a77f-7ab8cf195fcd/e4ad1a02-817a-4cce-9ee6-266c75a94756/9d30bcf3-6fd4-4ecd-bcd6-7dfab3ad93fc"
-          (reference "R57") (unit 1)
-        )
-      )
-    )
-  )
   (symbol (lib_id "Device:R") (at 114.3 168.91 0) (unit 1)
     (in_bom yes) (on_board yes) (dnp no)
@@
     )
   )
-  (symbol (lib_id "power:GND") (at 88.9 189.23 0) (unit 1)
-    (in_bom yes) (on_board yes) (dnp no) (fields_autoplaced)
-    (property "Reference" "#PWR0105" (at 88.9 195.58 0)
-      (effects (font (size 1.27 1.27)) hide)
-    )
-    (property "Value" "GND" (at 88.9 194.31 0)
-      (effects (font (size 1.27 1.27)))
-    )
-    (property "Footprint" "" (at 88.9 189.23 0)
-      (effects (font (size 1.27 1.27)) hide)
-    )
-    (property "Datasheet" "" (at 88.9 189.23 0)
-      (effects (font (size 1.27 1.27)) hide)
-    )
-    (pin "1")
-    (instances
-      (project "dongtam"
-        (path "/6833aec4-3d1d-4261-9b3e-f0452b565dd3/992d1183-82f3-4ab3-a77f-7ab8cf195fcd/e4ad1a02-817a-4cce-9ee6-266c75a94756/9d30bcf3-6fd4-4ecd-bcd6-7dfab3ad93fc"
-          (reference "#PWR0105") (unit 1)
-        )
-      )
-    )
-  )
-  (symbol (lib_id "Device:R") (at 88.9 184.15 0) (unit 1)
-    (in_bom yes) (on_board yes) (dnp no)
-    (property "Reference" "R58" (at 90.17 182.88 0)
-      (effects (font (size 1.27 1.27)) (justify left))
-    )
-    (property "Value" "1k" (at 90.17 185.42 0)
-      (effects (font (size 1.27 1.27)) (justify left))
-    )
-    (property "Footprint" "IVS_FOOTPRINTS:R0603" (at 87.122 184.15 90)
-      (effects (font (size 1.27 1.27)) hide)
-    )
-    (property "Datasheet" "~" (at 88.9 184.15 0)
-      (effects (font (size 1.27 1.27)) hide)
-    )
-    (pin "1")
-    (pin "2")
-    (instances
-      (project "dongtam"
-        (path "/6833aec4-3d1d-4261-9b3e-f0452b565dd3/992d1183-82f3-4ab3-a77f-7ab8cf195fcd/e4ad1a02-817a-4cce-9ee6-266c75a94756/9d30bcf3-6fd4-4ecd-bcd6-7dfab3ad93fc"
-          (reference "R58") (unit 1)
-        )
-      )
-    )
-  )
   (symbol (lib_id "power:GND") (at 81.28 30.48 0) (unit 1)
     (in_bom yes) (on_board yes) (dnp no)
@@
     )
   )
-  (symbol (lib_id "Device:R") (at 88.9 49.53 0) (unit 1)
-    (in_bom yes) (on_board yes) (dnp no)
-    (property "Reference" "R55" (at 90.17 48.26 0)
-      (effects (font (size 1.27 1.27)) (justify left))
-    )
-    (property "Value" "1k" (at 90.17 50.8 0)
-      (effects (font (size 1.27 1.27)) (justify left))
-    )
-    (property "Footprint" "IVS_FOOTPRINTS:R0603" (at 87.122 49.53 90)
-      (effects (font (size 1.27 1.27)) hide)
-    )
-    (property "Datasheet" "~" (at 88.9 49.53 0)
-      (effects (font (size 1.27 1.27)) hide)
-    )
-    (pin "1")
-    (pin "2")
-    (instances
-      (project "dongtam"
-        (path "/6833aec4-3d1d-4261-9b3e-f0452b565dd3/992d1183-82f3-4ab3-a77f-7ab8cf195fcd/e4ad1a02-817a-4cce-9ee6-266c75a94756/9d30bcf3-6fd4-4ecd-bcd6-7dfab3ad93fc"
-          (reference "R55") (unit 1)
-        )
-      )
-    )
-  )
-  (symbol (lib_id "power:GND") (at 88.9 143.51 0) (unit 1)
-    (in_bom yes) (on_board yes) (dnp no) (fields_autoplaced)
-    (property "Reference" "#PWR0104" (at 88.9 149.86 0)
-      (effects (font (size 1.27 1.27)) hide)
-    )
-    (property "Value" "GND" (at 88.9 148.59 0)
-      (effects (font (size 1.27 1.27)))
-    )
-    (property "Footprint" "" (at 88.9 143.51 0)
-      (effects (font (size 1.27 1.27)) hide)
-    )
-    (property "Datasheet" "" (at 88.9 143.51 0)
-      (effects (font (size 1.27 1.27)) hide)
-    )
-    (pin "1")
-    (instances
-      (project "dongtam"
-        (path "/6833aec4-3d1d-4261-9b3e-f0452b565dd3/992d1183-82f3-4ab3-a77f-7ab8cf195fcd/e4ad1a02-817a-4cce-9ee6-266c75a94756/9d30bcf3-6fd4-4ecd-bcd6-7dfab3ad93fc"
-          (reference "#PWR0104") (unit 1)
-        )
-      )
-    )
-  )
   (symbol (lib_id "Device:Q_NMOS_DGS") (at 64.77 167.64 0) (unit 1)
     (in_bom yes) (on_board yes) (dnp no)
@@
     )
   )
-  (symbol (lib_id "power:GND") (at 88.9 54.61 0) (unit 1)
-    (in_bom yes) (on_board yes) (dnp no) (fields_autoplaced)
-    (property "Reference" "#PWR0102" (at 88.9 60.96 0)
-      (effects (font (size 1.27 1.27)) hide)
-    )
-    (property "Value" "GND" (at 88.9 59.69 0)
-      (effects (font (size 1.27 1.27)))
-    )
-    (property "Footprint" "" (at 88.9 54.61 0)
-      (effects (font (size 1.27 1.27)) hide)
-    )
-    (property "Datasheet" "" (at 88.9 54.61 0)
-      (effects (font (size 1.27 1.27)) hide)
-    )
-    (pin "1")
-    (instances
-      (project "dongtam"
-        (path "/6833aec4-3d1d-4261-9b3e-f0452b565dd3/992d1183-82f3-4ab3-a77f-7ab8cf195fcd/e4ad1a02-817a-4cce-9ee6-266c75a94756/9d30bcf3-6fd4-4ecd-bcd6-7dfab3ad93fc"
-          (reference "#PWR0102") (unit 1)
-        )
-      )
-    )
-  )
   (symbol (lib_id "Device:Q_NMOS_DGS") (at 64.77 33.02 0) (unit 1)
     (in_bom yes) (on_board yes) (dnp no) (fields_autoplaced)
@@
         )
       )
-    )
-  )
-  (symbol (lib_id "power:GND") (at 88.9 100.33 0) (unit 1)
-    (in_bom yes) (on_board yes) (dnp no) (fields_autoplaced)
-    (property "Reference" "#PWR0103" (at 88.9 106.68 0)
-      (effects (font (size 1.27 1.27)) hide)
-    )
-    (property "Value" "GND" (at 88.9 105.41 0)
-      (effects (font (size 1.27 1.27)))
-    )
-    (property "Footprint" "" (at 88.9 100.33 0)
-      (effects (font (size 1.27 1.27)) hide)
-    )
-    (property "Datasheet" "" (at 88.9 100.33 0)
-      (effects (font (size 1.27 1.27)) hide)
-    )
-    (pin "1")
-    (instances
-      (project "dongtam"
-        (path "/6833aec4-3d1d-4261-9b3e-f0452b565dd3/992d1183-82f3-4ab3-a77f-7ab8cf195fcd/e4ad1a02-817a-4cce-9ee6-266c75a94756/9d30bcf3-6fd4-4ecd-bcd6-7dfab3ad93fc"
-          (reference "#PWR0103") (unit 1)
-        )
-      )

Commit message: layout PCB part 1
Parts:
- removed Q5, Q6, Q7, Q8: SI_2300, IVS_FOOTPRINTS:SOT23-3, symbol Device:Q_NMOS_DGS
- added Q4, Q5, Q6, Q7: N_Mosfet, IVS_FOOTPRINTS:SOT23-3, symbol IVS_SYMBOLS:N_Mosfet
Connections:
- net VAN5-: now also J8.8 (Pin_8), Q4.3 (D); no longer J8.2 (Pin_2)
- net VAN5_input: now also Q4.1 (G)
- net VAN6-: now also J8.6 (Pin_6), Q5.3 (D); no longer J8.4 (Pin_4)
- net VAN6_input: now also Q5.1 (G)
- net VAN7-: now also J8.4 (Pin_4), Q6.3 (D); no longer J8.6 (Pin_6)
- net VAN7_input: now also Q6.1 (G)
- net VAN8-: now also J8.2 (Pin_2), Q7.3 (D); no longer J8.8 (Pin_8)
- net VAN8_input: now also Q7.1 (G)
- net at R51.1, U12.3 (+): now also Q4.2 (S)
- net at R52.1, U12.5 (+): now also Q5.2 (S)
- net at R53.1, U12.10 (+): now also Q6.2 (S)
- net at R54.1, U12.12 (+): now also Q7.2 (S)
