File: Hardware/3_TL084IPT.kicad_sch (KiCad schematic)
At the start: 34 parts

Commit message: after merge dev
Parts:
- gave numbers to parts that had none: 30

Commit message: add R0603 footprint
Parts:
- C19: footprint (none) -> IVS_FOOTPRINTS:C0603
- R58, R59, R60, R61, R62, R63, R64, R65, R66, R67, R68, R69, R70, R71, R72, R73: footprint (none) -> IVS_FOOTPRINTS:R0603
Changed lines of the file:
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@@
       (effects (font (size 1.27 1.27)) (justify left))
     )
-    (property "Footprint" "" (id 2) (at 59.182 180.34 90)
+    (property "Footprint" "IVS_FOOTPRINTS:R0603" (id 2) (at 59.182 180.34 90)
       (effects (font (size 1.27 1.27)) hide)
     )
@@
       (effects (font (size 1.27 1.27)) (justify left))
     )
-    (property "Footprint" "" (id 2) (at 117.602 82.55 90)
+    (property "Footprint" "IVS_FOOTPRINTS:R0603" (id 2) (at 117.602 82.55 90)
       (effects (font (size 1.27 1.27)) hide)
     )
@@
       (effects (font (size 1.27 1.27)) (justify left))
     )
-    (property "Footprint" "" (id 2) (at 117.602 171.45 90)
+    (property "Footprint" "IVS_FOOTPRINTS:R0603" (id 2) (at 117.602 171.45 90)
       (effects (font (size 1.27 1.27)) hide)
     )
@@
       (effects (font (size 1.27 1.27)) (justify left))
     )
-    (property "Footprint" "" (id 2) (at 70.612 180.34 90)
+    (property "Footprint" "IVS_FOOTPRINTS:R0603" (id 2) (at 70.612 180.34 90)
       (effects (font (size 1.27 1.27)) hide)
     )
@@
       (effects (font (size 1.27 1.27)) (justify left))
     )
-    (property "Footprint" "" (id 2) (at 92.202 97.79 90)
+    (property "Footprint" "IVS_FOOTPRINTS:R0603" (id 2) (at 92.202 97.79 90)
       (effects (font (size 1.27 1.27)) hide)
     )
@@
       (effects (font (size 1.27 1.27)) (justify left))
     )
-    (property "Footprint" "" (id 2) (at 92.202 140.97 90)
+    (property "Footprint" "IVS_FOOTPRINTS:R0603" (id 2) (at 92.202 140.97 90)
       (effects (font (size 1.27 1.27)) hide)
     )
@@
       (effects (font (size 1.27 1.27)) (justify left))
     )
-    (property "Footprint" "" (id 2) (at 117.602 36.83 90)
+    (property "Footprint" "IVS_FOOTPRINTS:R0603" (id 2) (at 117.602 36.83 90)
       (effects (font (size 1.27 1.27)) hide)
     )
@@
       (effects (font (size 1.27 1.27)) (justify left))
     )
-    (property "Footprint" "" (id 2) (at 59.182 45.72 90)
+    (property "Footprint" "IVS_FOOTPRINTS:R0603" (id 2) (at 59.182 45.72 90)
       (effects (font (size 1.27 1.27)) hide)
     )
@@
       (effects (font (size 1.27 1.27)) (justify left))
     )
-    (property "Footprint" "" (id 2) (at 92.202 52.07 90)
+    (property "Footprint" "IVS_FOOTPRINTS:R0603" (id 2) (at 92.202 52.07 90)
       (effects (font (size 1.27 1.27)) hide)
     )
@@
       (effects (font (size 1.27 1.27)) (justify left))
     )
-    (property "Footprint" "" (id 2) (at 59.182 91.44 90)
+    (property "Footprint" "IVS_FOOTPRINTS:R0603" (id 2) (at 59.182 91.44 90)
       (effects (font (size 1.27 1.27)) hide)
     )
@@
       (effects (font (size 1.27 1.27)) (justify left))
     )
-    (property "Footprint" "" (id 2) (at 59.182 135.89 90)
+    (property "Footprint" "IVS_FOOTPRINTS:R0603" (id 2) (at 59.182 135.89 90)
       (effects (font (size 1.27 1.27)) hide)
     )
@@
       (effects (font (size 1.27 1.27)) (justify left))
     )
-    (property "Footprint" "" (id 2) (at 70.612 91.44 90)
+    (property "Footprint" "IVS_FOOTPRINTS:R0603" (id 2) (at 70.612 91.44 90)
       (effects (font (size 1.27 1.27)) hide)
     )
@@
       (effects (font (size 1.27 1.27)) (justify left))
     )
-    (property "Footprint" "" (id 2) (at 92.202 186.69 90)
+    (property "Footprint" "IVS_FOOTPRINTS:R0603" (id 2) (at 92.202 186.69 90)
       (effects (font (size 1.27 1.27)) hide)
     )
@@
       (effects (font (size 1.27 1.27)) (justify left))
     )
-    (property "Footprint" "" (id 2) (at 117.602 125.73 90)
+    (property "Footprint" "IVS_FOOTPRINTS:R0603" (id 2) (at 117.602 125.73 90)
       (effects (font (size 1.27 1.27)) hide)
     )
@@
       (effects (font (size 1.27 1.27)) (justify left))
     )
-    (property "Footprint" "" (id 2) (at 70.612 45.72 90)
+    (property "Footprint" "IVS_FOOTPRINTS:R0603" (id 2) (at 70.612 45.72 90)
       (effects (font (size 1.27 1.27)) hide)
     )
@@
       (effects (font (size 1.27 1.27)) (justify left))
     )
-    (property "Footprint" "" (id 2) (at 87.3252 33.02 0)
+    (property "Footprint" "IVS_FOOTPRINTS:C0603" (id 2) (at 87.3252 33.02 0)
       (effects (font (size 1.27 1.27)) hide)
     )
@@
       (effects (font (size 1.27 1.27)) (justify left))
     )
-    (property "Footprint" "" (id 2) (at 70.612 135.89 90)
-      (effects (font (size 1.27 1.27)) hide)
-    )
+    (property "Footprint" "IVS_FOOTPRINTS:R0603" (id 2) (at 70.612 135.89 90)
+      (effects (font (size 1.27 1.27)) hide)
+    )

Commit message: fix MCP41010, fix symbol output header
Parts:
- J14: renamed from J12; symbol Connector:Conn_01x02_Male -> Connector:Screw_Terminal_01x02
- J15: renamed from J13; symbol Connector:Conn_01x02_Male -> Connector:Screw_Terminal_01x02
- J16: renamed from J14; symbol Connector:Conn_01x02_Male -> Connector:Screw_Terminal_01x02
- J17: renamed from J15; symbol Connector:Conn_01x02_Male -> Connector:Screw_Terminal_01x02
- R67: renamed from R62; footprint IVS_FOOTPRINTS:R0603 -> Resistor_SMD:R_0805_2012Metric
- R68: renamed from R63; footprint IVS_FOOTPRINTS:R0603 -> Resistor_SMD:R_0805_2012Metric
- R69: renamed from R64; footprint IVS_FOOTPRINTS:R0603 -> Resistor_SMD:R_0805_2012Metric
- R70: renamed from R65; footprint IVS_FOOTPRINTS:R0603 -> Resistor_SMD:R_0805_2012Metric
- renumbered C19 to C30, R58 to R63, R59 to R64, R60 to R65, R61 to R66, R66 to R71, R67 to R72, R68 to R73, R69 to R74, R70 to R75, R71 to R76, R72 to R77, R73 to R78, U12 to U13
Connections:
- net PA0_MCP41010 renamed PW0_MCP41

Commit message: add footprint
Parts:
- removed J14: VAN10, symbol Connector:Screw_Terminal_01x02
- removed J15: VAN11, symbol Connector:Screw_Terminal_01x02
- removed J16: VAN12, symbol Connector:Screw_Terminal_01x02
- removed J17: VAN9, symbol Connector:Screw_Terminal_01x02
- added J?: Screw_Terminal_01x08, IVS_FOOTPRINTS:HT-3.96mm, symbol Connector:Screw_Terminal_01x08
Connections:
- net +24V: now also J?.1 (Pin_1), J?.3 (Pin_3), J?.5 (Pin_5), J?.7 (Pin_7)
- net VAN9-: now reaches D16.1, Q9.1 (D)
- net VAN9-: now also J?.2 (Pin_2)
- net VAN10-: now reaches D17.1, Q10.1 (D)
- net VAN10-: now also J?.4 (Pin_4)
- net VAN12-: now reaches D19.1, Q12.1 (D)
- net VAN12-: now also J?.8 (Pin_8)
- net VAN11-: now reaches D18.1, Q11.1 (D)
- net VAN11-: now also J?.6 (Pin_6)
Changed lines of the file:
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@@
     (stroke (width 0) (type default) (color 0 0 0 0))
+  )
+  (label "VAN12-" (at 55.88 161.29 0)
+    (effects (font (size 1.27 1.27)) (justify left bottom))
+  )
+  (label "VAN11+" (at 24.765 116.205 0)
+    (effects (font (size 1.27 1.27)) (justify left bottom))
+  )
+  (label "VAN12+" (at 55.88 158.75 0)
+    (effects (font (size 1.27 1.27)) (justify left bottom))
+  )
+  (label "VAN10+" (at 24.765 111.125 0)
+    (effects (font (size 1.27 1.27)) (justify left bottom))
+  )
+  (label "VAN9-" (at 24.765 108.585 0)
+    (effects (font (size 1.27 1.27)) (justify left bottom))
+  )
+  (label "VAN11-" (at 24.765 118.745 0)
+    (effects (font (size 1.27 1.27)) (justify left bottom))
+  )
+  (label "VAN11+" (at 55.88 114.3 0)
+    (effects (font (size 1.27 1.27)) (justify left bottom))
+  )
+  (label "VAN10-" (at 24.765 113.665 0)
+    (effects (font (size 1.27 1.27)) (justify left bottom))
+  )
+  (label "VAN9-" (at 58.42 26.67 0)
+    (effects (font (size 1.27 1.27)) (justify left bottom))
+  )
+  (label "VAN12-" (at 24.765 123.825 0)
+    (effects (font (size 1.27 1.27)) (justify left bottom))
+  )
+  (label "VAN9+" (at 24.765 106.045 0)
+    (effects (font (size 1.27 1.27)) (justify left bottom))
+  )
+  (label "VAN9+" (at 58.42 24.13 0)
+    (effects (font (size 1.27 1.27)) (justify left bottom))
+  )
+  (label "VAN11-" (at 55.88 116.84 0)
+    (effects (font (size 1.27 1.27)) (justify left bottom))
+  )
+  (label "VAN10-" (at 54.61 72.39 0)
+    (effects (font (size 1.27 1.27)) (justify left bottom))
+  )
+  (label "VAN12+" (at 24.765 121.285 0)
+    (effects (font (size 1.27 1.27)) (justify left bottom))
+  )
+  (label "VAN10+" (at 54.61 69.85 0)
+    (effects (font (size 1.27 1.27)) (justify left bottom))
   )
   (hierarchical_label "VAN12_output" (shape output) (at 124.46 179.07 0)
@@
     (pin "1")
   )
-  (symbol (lib_id "Connector:Screw_Terminal_01x02") (at 50.8 158.75 0) (mirror y) (unit 1)
-    (in_bom yes) (on_board yes) (fields_autoplaced)
-    (property "Reference" "J16" (id 0) (at 50.8 152.4 0))
-    (property "Value" "VAN12" (id 1) (at 50.8 154.94 0))
-    (property "Footprint" "" (id 2) (at 50.8 158.75 0)
-      (effects (font (size 1.27 1.27)) hide)
-    )
-    (property "Datasheet" "~" (id 3) (at 50.8 158.75 0)
-      (effects (font (size 1.27 1.27)) hide)
-    )
-    (pin "1")
-    (pin "2")
-  )
   (symbol (lib_id "power:GND") (at 93.98 146.05 0) (unit 1)
     (in_bom yes) (on_board yes) (fields_autoplaced)
@@
     (pin "2")
   )
-  (symbol (lib_id "Connector:Screw_Terminal_01x02") (at 53.34 24.13 0) (mirror y) (unit 1)
-    (in_bom yes) (on_board yes) (fields_autoplaced)
-    (property "Reference" "J17" (id 0) (at 53.34 17.78 0))
-    (property "Value" "VAN9" (id 1) (at 53.34 20.32 0))
-    (property "Footprint" "" (id 2) (at 53.34 24.13 0)
-      (effects (font (size 1.27 1.27)) hide)
-    )
-    (property "Datasheet" "~" (id 3) (at 53.34 24.13 0)
-      (effects (font (size 1.27 1.27)) hide)
-    )
-    (pin "1")
-    (pin "2")
-  )
   (symbol (lib_id "Device:Q_NMOS_DGS") (at 69.85 125.73 0) (unit 1)
     (in_bom yes) (on_board yes)
@@
     )
     (property "Datasheet" "~" (id 3) (at 119.38 36.83 0)
-      (effects (font (size 1.27 1.27)) hide)
-    )
-    (pin "1")
-    (pin "2")
-  )
-  (symbol (lib_id "Connector:Screw_Terminal_01x02") (at 49.53 69.85 0) (mirror y) (unit 1)
-    (in_bom yes) (on_board yes) (fields_autoplaced)
-    (property "Reference" "J14" (id 0) (at 49.53 63.5 0))
-    (property "Value" "VAN10" (id 1) (at 49.53 66.04 0))
-    (property "Footprint" "" (id 2) (at 49.53 69.85 0)
-      (effects (font (size 1.27 1.27)) hide)
-    )
-    (property "Datasheet" "~" (id 3) (at 49.53 69.85 0)
       (effects (font (size 1.27 1.27)) hide)
     )
@@
     (pin "1")
   )
+  (symbol (lib_id "Connector:Screw_Terminal_01x08") (at 19.685 113.665 0) (mirror y) (unit 1)
+    (in_bom yes) (on_board yes) (fields_autoplaced)
+    (property "Reference" "J?" (id 0) (at 19.685 99.695 0))
+    (property "Value" "Screw_Terminal_01x08" (id 1) (at 19.685 102.235 0))
+    (property "Footprint" "IVS_FOOTPRINTS:HT-3.96mm" (id 2) (at 19.685 113.665 0)
+      (effects (font (size 1.27 1.27)) hide)
+    )
+    (property "Datasheet" "~" (id 3) (at 19.685 113.665 0)
+      (effects (font (size 1.27 1.27)) hide)
+    )
+    (pin "1")
+    (pin "2")
+    (pin "3")
+    (pin "4")
+    (pin "5")
+    (pin "6")
+    (pin "7")
+    (pin "8")
+  )
   (symbol (lib_id "Device:R") (at 93.98 186.69 0) (unit 1)
     (in_bom yes) (on_board yes)
@@
     (pin "1")
   )
-  (symbol (lib_id "Connector:Screw_Terminal_01x02") (at 50.8 114.3 0) (mirror y) (unit 1)
-    (in_bom yes) (on_board yes) (fields_autoplaced)
-    (property "Reference" "J15" (id 0) (at 50.8 107.95 0))
-    (property "Value" "VAN11" (id 1) (at 50.8 110.49 0))
-    (property "Footprint" "" (id 2) (at 50.8 114.3 0)
-      (effects (font (size 1.27 1.27)) hide)
-    )
-    (property "Datasheet" "~" (id 3) (at 50.8 114.3 0)
-      (effects (font (size 1.27 1.27)) hide)
-    )
-    (pin "1")
-    (pin "2")
-  )
   (symbol (lib_id "IVS_SYMBOL_DIR:D_Diode") (at 72.39 158.75 270) (unit 1)

Commit message: add all footprint
Parts:
- gave numbers to parts that had none: 1
Changed lines of the file:
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@@
   (symbol (lib_id "power:+24V") (at 72.39 109.22 0) (unit 1)
     (in_bom yes) (on_board yes) (fields_autoplaced)
-    (property "Reference" "#PWR0111" (id 0) (at 72.39 113.03 0)
+    (property "Reference" "#PWR0115" (id 0) (at 72.39 113.03 0)
       (effects (font (size 1.27 1.27)) hide)
     )
@@
   (symbol (lib_id "power:GND") (at 72.39 186.69 0) (unit 1)
     (in_bom yes) (on_board yes) (fields_autoplaced)
-    (property "Reference" "#PWR0114" (id 0) (at 72.39 193.04 0)
+    (property "Reference" "#PWR0118" (id 0) (at 72.39 193.04 0)
       (effects (font (size 1.27 1.27)) hide)
     )
@@
   (symbol (lib_id "power:GND") (at 72.39 97.79 0) (unit 1)
     (in_bom yes) (on_board yes) (fields_autoplaced)
-    (property "Reference" "#PWR0110" (id 0) (at 72.39 104.14 0)
+    (property "Reference" "#PWR0114" (id 0) (at 72.39 104.14 0)
       (effects (font (size 1.27 1.27)) hide)
     )
@@
   (symbol (lib_id "power:+24V") (at 72.39 64.77 0) (unit 1)
     (in_bom yes) (on_board yes) (fields_autoplaced)
-    (property "Reference" "#PWR0109" (id 0) (at 72.39 68.58 0)
+    (property "Reference" "#PWR0113" (id 0) (at 72.39 68.58 0)
       (effects (font (size 1.27 1.27)) hide)
     )
@@
   (symbol (lib_id "power:+3V3") (at 119.38 31.75 0) (unit 1)
     (in_bom yes) (on_board yes) (fields_autoplaced)
-    (property "Reference" "#PWR0122" (id 0) (at 119.38 35.56 0)
+    (property "Reference" "#PWR0126" (id 0) (at 119.38 35.56 0)
       (effects (font (size 1.27 1.27)) hide)
     )
@@
   (symbol (lib_id "power:GND") (at 86.36 33.02 0) (unit 1)
     (in_bom yes) (on_board yes)
-    (property "Reference" "#PWR0116" (id 0) (at 86.36 39.37 0)
+    (property "Reference" "#PWR0120" (id 0) (at 86.36 39.37 0)
       (effects (font (size 1.27 1.27)) hide)
     )
@@
   (symbol (lib_id "power:+3V3") (at 119.38 166.37 0) (unit 1)
     (in_bom yes) (on_board yes) (fields_autoplaced)
-    (property "Reference" "#PWR0125" (id 0) (at 119.38 170.18 0)
+    (property "Reference" "#PWR0129" (id 0) (at 119.38 170.18 0)
       (effects (font (size 1.27 1.27)) hide)
     )
@@
   (symbol (lib_id "power:+24V") (at 72.39 153.67 0) (unit 1)
     (in_bom yes) (on_board yes) (fields_autoplaced)
-    (property "Reference" "#PWR0113" (id 0) (at 72.39 157.48 0)
+    (property "Reference" "#PWR0117" (id 0) (at 72.39 157.48 0)
       (effects (font (size 1.27 1.27)) hide)
     )
@@
   (symbol (lib_id "power:GND") (at 93.98 57.15 0) (unit 1)
     (in_bom yes) (on_board yes) (fields_autoplaced)
-    (property "Reference" "#PWR0117" (id 0) (at 93.98 63.5 0)
+    (property "Reference" "#PWR0121" (id 0) (at 93.98 63.5 0)
       (effects (font (size 1.27 1.27)) hide)
     )
@@
   (symbol (lib_id "power:GND") (at 93.98 146.05 0) (unit 1)
     (in_bom yes) (on_board yes) (fields_autoplaced)
-    (property "Reference" "#PWR0119" (id 0) (at 93.98 152.4 0)
+    (property "Reference" "#PWR0123" (id 0) (at 93.98 152.4 0)
       (effects (font (size 1.27 1.27)) hide)
     )
@@
   (symbol (lib_id "power:GND") (at 93.98 102.87 0) (unit 1)
     (in_bom yes) (on_board yes) (fields_autoplaced)
-    (property "Reference" "#PWR0118" (id 0) (at 93.98 109.22 0)
+    (property "Reference" "#PWR0122" (id 0) (at 93.98 109.22 0)
       (effects (font (size 1.27 1.27)) hide)
     )
@@
   (symbol (lib_id "power:+24V") (at 72.39 20.32 0) (unit 1)
     (in_bom yes) (on_board yes) (fields_autoplaced)
-    (property "Reference" "#PWR0107" (id 0) (at 72.39 24.13 0)
+    (property "Reference" "#PWR0111" (id 0) (at 72.39 24.13 0)
       (effects (font (size 1.27 1.27)) hide)
     )
@@
   (symbol (lib_id "power:+3V3") (at 119.38 120.65 0) (unit 1)
     (in_bom yes) (on_board yes) (fields_autoplaced)
-    (property "Reference" "#PWR0124" (id 0) (at 119.38 124.46 0)
+    (property "Reference" "#PWR0128" (id 0) (at 119.38 124.46 0)
       (effects (font (size 1.27 1.27)) hide)
     )
@@
   (symbol (lib_id "power:GND") (at 72.39 52.07 0) (unit 1)
     (in_bom yes) (on_board yes) (fields_autoplaced)
-    (property "Reference" "#PWR0108" (id 0) (at 72.39 58.42 0)
+    (property "Reference" "#PWR0112" (id 0) (at 72.39 58.42 0)
       (effects (font (size 1.27 1.27)) hide)
     )
@@
   (symbol (lib_id "power:GND") (at 72.39 142.24 0) (unit 1)
     (in_bom yes) (on_board yes) (fields_autoplaced)
-    (property "Reference" "#PWR0112" (id 0) (at 72.39 148.59 0)
+    (property "Reference" "#PWR0116" (id 0) (at 72.39 148.59 0)
       (effects (font (size 1.27 1.27)) hide)
     )
@@
   (symbol (lib_id "power:GND") (at 107.95 25.4 0) (unit 1)
     (in_bom yes) (on_board yes) (fields_autoplaced)
-    (property "Reference" "#PWR0121" (id 0) (at 107.95 31.75 0)
+    (property "Reference" "#PWR0125" (id 0) (at 107.95 31.75 0)
       (effects (font (size 1.27 1.27)) hide)
     )
@@
   (symbol (lib_id "Connector:Screw_Terminal_01x08") (at 19.685 113.665 0) (mirror y) (unit 1)
     (in_bom yes) (on_board yes) (fields_autoplaced)
-    (property "Reference" "J?" (id 0) (at 19.685 99.695 0))
+    (property "Reference" "J9" (id 0) (at 19.685 99.695 0))
     (property "Value" "Screw_Terminal_01x08" (id 1) (at 19.685 102.235 0))
     (property "Footprint" "IVS_FOOTPRINTS:HT-3.96mm" (id 2) (at 19.685 113.665 0)
@@
   (symbol (lib_id "power:+3V3") (at 86.36 25.4 0) (unit 1)
     (in_bom yes) (on_board yes) (fields_autoplaced)
-    (property "Reference" "#PWR0115" (id 0) (at 86.36 29.21 0)
+    (property "Reference" "#PWR0119" (id 0) (at 86.36 29.21 0)
       (effects (font (size 1.27 1.27)) hide)
     )
@@
   (symbol (lib_id "power:GND") (at 93.98 191.77 0) (unit 1)
     (in_bom yes) (on_board yes) (fields_autoplaced)
-    (property "Reference" "#PWR0120" (id 0) (at 93.98 198.12 0)
+    (property "Reference" "#PWR0124" (id 0) (at 93.98 198.12 0)
       (effects (font (size 1.27 1.27)) hide)
     )
@@
   (symbol (lib_id "power:+3V3") (at 119.38 77.47 0) (unit 1)
     (in_bom yes) (on_board yes) (fields_autoplaced)
-    (property "Reference" "#PWR0123" (id 0) (at 119.38 81.28 0)
-      (effects (font (size 1.27 1.27)) hide)
-    )
+    (property "Reference" "#PWR0127" (id 0) (at 119.38 81.28 0)
+      (effects (font (size 1.27 1.27)) hide)
+    )
