File: Hardware/3_TL084IPT.kicad_sch (KiCad schematic)
At the start: 27 parts, among them J9 Screw_Terminal_01x08, Q10 SI_2300, Q11 SI_2300, Q12 SI_2300, Q9 SI_2300, U13 TL084

Commit message: add shematics MVA
Parts:
- removed R71, R72, R73, R74: 1k, IVS_FOOTPRINTS:R0603, symbol Device:R
Changed lines of the file:
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@@
-    (stroke (width 0) (type default))
-  )
-  (wire (pts (xy 93.98 102.87) (xy 93.98 101.6))
     (stroke (width 0) (type default))
   )
@@
     (stroke (width 0) (type default))
   )
-  (wire (pts (xy 93.98 48.26) (xy 93.98 46.99))
-    (stroke (width 0) (type default))
-  )
   (wire (pts (xy 111.76 44.45) (xy 119.38 44.45))
     (stroke (width 0) (type default))
@@
     (stroke (width 0) (type default))
   )
-  (wire (pts (xy 93.98 57.15) (xy 93.98 55.88))
-    (stroke (width 0) (type default))
-  )
   (wire (pts (xy 119.38 121.92) (xy 119.38 120.65))
     (stroke (width 0) (type default))
@@
     (stroke (width 0) (type default))
   )
-  (wire (pts (xy 93.98 137.16) (xy 93.98 135.89))
-    (stroke (width 0) (type default))
-  )
   (wire (pts (xy 60.96 49.53) (xy 72.39 49.53))
     (stroke (width 0) (type default))
@@
     (stroke (width 0) (type default))
   )
-  (wire (pts (xy 93.98 93.98) (xy 93.98 92.71))
-    (stroke (width 0) (type default))
-  )
   (wire (pts (xy 60.96 114.3) (xy 60.96 110.49))
     (stroke (width 0) (type default))
@@
     (stroke (width 0) (type default))
   )
-  (wire (pts (xy 93.98 146.05) (xy 93.98 144.78))
-    (stroke (width 0) (type default))
-  )
   (wire (pts (xy 119.38 167.64) (xy 119.38 166.37))
     (stroke (width 0) (type default))
@@
     (stroke (width 0) (type default))
   )
-  (wire (pts (xy 93.98 191.77) (xy 93.98 190.5))
-    (stroke (width 0) (type default))
-  )
   (wire (pts (xy 72.39 95.25) (xy 72.39 97.79))
     (stroke (width 0) (type default))
@@
   )
   (wire (pts (xy 119.38 86.36) (xy 119.38 90.17))
-    (stroke (width 0) (type default))
-  )
-  (wire (pts (xy 93.98 182.88) (xy 93.98 181.61))
     (stroke (width 0) (type default))
   )
@@
     )
   )
-  (symbol (lib_id "power:GND") (at 93.98 57.15 0) (unit 1)
-    (in_bom yes) (on_board yes) (dnp no) (fields_autoplaced)
-    (property "Reference" "#PWR0121" (at 93.98 63.5 0)
-      (effects (font (size 1.27 1.27)) hide)
-    )
-    (property "Value" "GND" (at 93.98 62.23 0)
-      (effects (font (size 1.27 1.27)))
-    )
-    (property "Footprint" "" (at 93.98 57.15 0)
-      (effects (font (size 1.27 1.27)) hide)
-    )
-    (property "Datasheet" "" (at 93.98 57.15 0)
-      (effects (font (size 1.27 1.27)) hide)
-    )
-    (pin "1")
-    (instances
-      (project "dongtam"
-        (path "/6833aec4-3d1d-4261-9b3e-f0452b565dd3/992d1183-82f3-4ab3-a77f-7ab8cf195fcd/e4ad1a02-817a-4cce-9ee6-266c75a94756/4a4886c5-9f9e-4e2f-a5aa-810911de4343"
-          (reference "#PWR0121") (unit 1)
-        )
-      )
-    )
-  )
-  (symbol (lib_id "power:GND") (at 93.98 146.05 0) (unit 1)
-    (in_bom yes) (on_board yes) (dnp no) (fields_autoplaced)
-    (property "Reference" "#PWR0123" (at 93.98 152.4 0)
-      (effects (font (size 1.27 1.27)) hide)
-    )
-    (property "Value" "GND" (at 93.98 151.13 0)
-      (effects (font (size 1.27 1.27)))
-    )
-    (property "Footprint" "" (at 93.98 146.05 0)
-      (effects (font (size 1.27 1.27)) hide)
-    )
-    (property "Datasheet" "" (at 93.98 146.05 0)
-      (effects (font (size 1.27 1.27)) hide)
-    )
-    (pin "1")
-    (instances
-      (project "dongtam"
-        (path "/6833aec4-3d1d-4261-9b3e-f0452b565dd3/992d1183-82f3-4ab3-a77f-7ab8cf195fcd/e4ad1a02-817a-4cce-9ee6-266c75a94756/4a4886c5-9f9e-4e2f-a5aa-810911de4343"
-          (reference "#PWR0123") (unit 1)
-        )
-      )
-    )
-  )
-  (symbol (lib_id "Device:R") (at 93.98 97.79 0) (unit 1)
-    (in_bom yes) (on_board yes) (dnp no)
-    (property "Reference" "R72" (at 95.25 96.52 0)
-      (effects (font (size 1.27 1.27)) (justify left))
-    )
-    (property "Value" "1k" (at 95.25 99.06 0)
-      (effects (font (size 1.27 1.27)) (justify left))
-    )
-    (property "Footprint" "IVS_FOOTPRINTS:R0603" (at 92.202 97.79 90)
-      (effects (font (size 1.27 1.27)) hide)
-    )
-    (property "Datasheet" "~" (at 93.98 97.79 0)
-      (effects (font (size 1.27 1.27)) hide)
-    )
-    (pin "1")
-    (pin "2")
-    (instances
-      (project "dongtam"
-        (path "/6833aec4-3d1d-4261-9b3e-f0452b565dd3/992d1183-82f3-4ab3-a77f-7ab8cf195fcd/e4ad1a02-817a-4cce-9ee6-266c75a94756/4a4886c5-9f9e-4e2f-a5aa-810911de4343"
-          (reference "R72") (unit 1)
-        )
-      )
-    )
-  )
-  (symbol (lib_id "Device:R") (at 93.98 140.97 0) (unit 1)
-    (in_bom yes) (on_board yes) (dnp no)
-    (property "Reference" "R73" (at 95.25 139.7 0)
-      (effects (font (size 1.27 1.27)) (justify left))
-    )
-    (property "Value" "1k" (at 95.25 142.24 0)
-      (effects (font (size 1.27 1.27)) (justify left))
-    )
-    (property "Footprint" "IVS_FOOTPRINTS:R0603" (at 92.202 140.97 90)
-      (effects (font (size 1.27 1.27)) hide)
-    )
-    (property "Datasheet" "~" (at 93.98 140.97 0)
-      (effects (font (size 1.27 1.27)) hide)
-    )
-    (pin "1")
-    (pin "2")
-    (instances
-      (project "dongtam"
-        (path "/6833aec4-3d1d-4261-9b3e-f0452b565dd3/992d1183-82f3-4ab3-a77f-7ab8cf195fcd/e4ad1a02-817a-4cce-9ee6-266c75a94756/4a4886c5-9f9e-4e2f-a5aa-810911de4343"
-          (reference "R73") (unit 1)
-        )
-      )
-    )
-  )
   (symbol (lib_id "Device:Q_NMOS_DGS") (at 69.85 125.73 0) (unit 1)
     (in_bom yes) (on_board yes) (dnp no)
@@
         (path "/6833aec4-3d1d-4261-9b3e-f0452b565dd3/992d1183-82f3-4ab3-a77f-7ab8cf195fcd/e4ad1a02-817a-4cce-9ee6-266c75a94756/4a4886c5-9f9e-4e2f-a5aa-810911de4343"
           (reference "Q11") (unit 1)
-        )
-      )
-    )
-  )
-  (symbol (lib_id "power:GND") (at 93.98 102.87 0) (unit 1)
-    (in_bom yes) (on_board yes) (dnp no) (fields_autoplaced)
-    (property "Reference" "#PWR0122" (at 93.98 109.22 0)
-      (effects (font (size 1.27 1.27)) hide)
-    )
-    (property "Value" "GND" (at 93.98 107.95 0)
-      (effects (font (size 1.27 1.27)))
-    )
-    (property "Footprint" "" (at 93.98 102.87 0)
-      (effects (font (size 1.27 1.27)) hide)
-    )
-    (property "Datasheet" "" (at 93.98 102.87 0)
-      (effects (font (size 1.27 1.27)) hide)
-    )
-    (pin "1")
-    (instances
-      (project "dongtam"
-        (path "/6833aec4-3d1d-4261-9b3e-f0452b565dd3/992d1183-82f3-4ab3-a77f-7ab8cf195fcd/e4ad1a02-817a-4cce-9ee6-266c75a94756/4a4886c5-9f9e-4e2f-a5aa-810911de4343"
-          (reference "#PWR0122") (unit 1)
         )
       )
@@
     )
   )
-  (symbol (lib_id "Device:R") (at 93.98 52.07 0) (unit 1)
-    (in_bom yes) (on_board yes) (dnp no)
-    (property "Reference" "R71" (at 95.25 50.8 0)
-      (effects (font (size 1.27 1.27)) (justify left))
-    )
-    (property "Value" "1k" (at 95.25 53.34 0)
-      (effects (font (size 1.27 1.27)) (justify left))
-    )
-    (property "Footprint" "IVS_FOOTPRINTS:R0603" (at 92.202 52.07 90)
-      (effects (font (size 1.27 1.27)) hide)
-    )
-    (property "Datasheet" "~" (at 93.98 52.07 0)
-      (effects (font (size 1.27 1.27)) hide)
-    )
-    (pin "1")
-    (pin "2")
-    (instances
-      (project "dongtam"
-        (path "/6833aec4-3d1d-4261-9b3e-f0452b565dd3/992d1183-82f3-4ab3-a77f-7ab8cf195fcd/e4ad1a02-817a-4cce-9ee6-266c75a94756/4a4886c5-9f9e-4e2f-a5aa-810911de4343"
-          (reference "R71") (unit 1)
-        )
-      )
-    )
-  )
   (symbol (lib_id "Amplifier_Operational:TL084") (at 104.14 44.45 0) (unit 1)
     (in_bom yes) (on_board yes) (dnp no) (fields_autoplaced)
@@
     )
   )
-  (symbol (lib_id "Device:R") (at 93.98 186.69 0) (unit 1)
-    (in_bom yes) (on_board yes) (dnp no)
-    (property "Reference" "R74" (at 95.25 185.42 0)
-      (effects (font (size 1.27 1.27)) (justify left))
-    )
-    (property "Value" "1k" (at 95.25 187.96 0)
-      (effects (font (size 1.27 1.27)) (justify left))
-    )
-    (property "Footprint" "IVS_FOOTPRINTS:R0603" (at 92.202 186.69 90)
-      (effects (font (size 1.27 1.27)) hide)
-    )
-    (property "Datasheet" "~" (at 93.98 186.69 0)
-      (effects (font (size 1.27 1.27)) hide)
-    )
-    (pin "1")
-    (pin "2")
-    (instances
-      (project "dongtam"
-        (path "/6833aec4-3d1d-4261-9b3e-f0452b565dd3/992d1183-82f3-4ab3-a77f-7ab8cf195fcd/e4ad1a02-817a-4cce-9ee6-266c75a94756/4a4886c5-9f9e-4e2f-a5aa-810911de4343"
-          (reference "R74") (unit 1)
-        )
-      )
-    )
-  )
   (symbol (lib_id "Device:R") (at 119.38 125.73 0) (unit 1)
     (in_bom yes) (on_board yes) (dnp no)
@@
         )
       )
-    )
-  )
-  (symbol (lib_id "power:GND") (at 93.98 191.77 0) (unit 1)
-    (in_bom yes) (on_board yes) (dnp no) (fields_autoplaced)
-    (property "Reference" "#PWR0124" (at 93.98 198.12 0)
-      (effects (font (size 1.27 1.27)) hide)
-    )
-    (property "Value" "GND" (at 93.98 196.85 0)
-      (effects (font (size 1.27 1.27)))
-    )
-    (property "Footprint" "" (at 93.98 191.77 0)
-      (effects (font (size 1.27 1.27)) hide)
-    )
-    (property "Datasheet" "" (at 93.98 191.77 0)
-      (effects (font (size 1.27 1.27)) hide)
-    )
-    (pin "1")
-    (instances
-      (project "dongtam"
-        (path "/6833aec4-3d1d-4261-9b3e-f0452b565dd3/992d1183-82f3-4ab3-a77f-7ab8cf195fcd/e4ad1a02-817a-4cce-9ee6-266c75a94756/4a4886c5-9f9e-4e2f-a5aa-810911de4343"
-          (reference "#PWR0124") (unit 1)
-        )
-      )

Commit message: layout PCB part 1
Parts:
- removed Q10, Q11, Q12, Q9: SI_2300, IVS_FOOTPRINTS:SOT23-3, symbol Device:Q_NMOS_DGS
- added Q10, Q11, Q8, Q9: N_Mosfet, IVS_FOOTPRINTS:SOT23-3, symbol IVS_SYMBOLS:N_Mosfet
Connections:
- net VAN10-: now also J9.6 (Pin_6), Q9.3 (D); no longer J9.4 (Pin_4)
- net VAN10_input: now also Q9.1 (G)
- net VAN11-: now also J9.4 (Pin_4), Q10.3 (D); no longer J9.6 (Pin_6)
- net VAN11_input: now also Q10.1 (G)
- net VAN12-: now also J9.2 (Pin_2), Q11.3 (D); no longer J9.8 (Pin_8)
- net VAN12_input: now also Q11.1 (G)
- net VAN9-: now also J9.8 (Pin_8), Q8.3 (D); no longer J9.2 (Pin_2)
- net VAN9_input: now also Q8.1 (G)
- net at R68.1, U13.5 (+): now also Q9.2 (S)
- net at R70.1, U13.12 (+): now also Q11.2 (S)
- net at R69.1, U13.10 (+): now also Q10.2 (S)
- net at R67.1, U13.3 (+): now also Q8.2 (S)
