File: Hardware/4_TL084IPT.kicad_sch (KiCad schematic)
At the start: 27 parts, among them Q13 SI_2300, Q14 SI_2300, Q15 SI_2300, Q16 SI_2300, U14 TL084

Commit message: add all footprint
Parts:
- gave numbers to parts that had none: 1
Changed lines of the file:
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@@
   (symbol (lib_id "power:GND") (at 88.9 100.33 0) (unit 1)
     (in_bom yes) (on_board yes) (fields_autoplaced)
-    (property "Reference" "#PWR0129" (id 0) (at 88.9 106.68 0)
+    (property "Reference" "#PWR0133" (id 0) (at 88.9 106.68 0)
       (effects (font (size 1.27 1.27)) hide)
     )
@@
   (symbol (lib_id "power:+3V3") (at 135.89 123.19 0) (unit 1)
     (in_bom yes) (on_board yes) (fields_autoplaced)
-    (property "Reference" "#PWR0143" (id 0) (at 135.89 127 0)
+    (property "Reference" "#PWR0147" (id 0) (at 135.89 127 0)
       (effects (font (size 1.27 1.27)) hide)
     )
@@
   (symbol (lib_id "power:GND") (at 124.46 27.94 0) (unit 1)
     (in_bom yes) (on_board yes) (fields_autoplaced)
-    (property "Reference" "#PWR0140" (id 0) (at 124.46 34.29 0)
+    (property "Reference" "#PWR0144" (id 0) (at 124.46 34.29 0)
       (effects (font (size 1.27 1.27)) hide)
     )
@@
   (symbol (lib_id "power:+3V3") (at 135.89 80.01 0) (unit 1)
     (in_bom yes) (on_board yes) (fields_autoplaced)
-    (property "Reference" "#PWR0142" (id 0) (at 135.89 83.82 0)
+    (property "Reference" "#PWR0146" (id 0) (at 135.89 83.82 0)
       (effects (font (size 1.27 1.27)) hide)
     )
@@
   (symbol (lib_id "power:GND") (at 110.49 148.59 0) (unit 1)
     (in_bom yes) (on_board yes) (fields_autoplaced)
-    (property "Reference" "#PWR0138" (id 0) (at 110.49 154.94 0)
+    (property "Reference" "#PWR0142" (id 0) (at 110.49 154.94 0)
       (effects (font (size 1.27 1.27)) hide)
     )
@@
   (symbol (lib_id "power:GND") (at 88.9 144.78 0) (unit 1)
     (in_bom yes) (on_board yes) (fields_autoplaced)
-    (property "Reference" "#PWR0131" (id 0) (at 88.9 151.13 0)
+    (property "Reference" "#PWR0135" (id 0) (at 88.9 151.13 0)
       (effects (font (size 1.27 1.27)) hide)
     )
@@
   (symbol (lib_id "power:GND") (at 110.49 105.41 0) (unit 1)
     (in_bom yes) (on_board yes) (fields_autoplaced)
-    (property "Reference" "#PWR0137" (id 0) (at 110.49 111.76 0)
+    (property "Reference" "#PWR0141" (id 0) (at 110.49 111.76 0)
       (effects (font (size 1.27 1.27)) hide)
     )
@@
   (symbol (lib_id "power:GND") (at 102.87 35.56 0) (unit 1)
     (in_bom yes) (on_board yes)
-    (property "Reference" "#PWR0135" (id 0) (at 102.87 41.91 0)
+    (property "Reference" "#PWR0139" (id 0) (at 102.87 41.91 0)
       (effects (font (size 1.27 1.27)) hide)
     )
@@
   (symbol (lib_id "power:+24V") (at 88.9 67.31 0) (unit 1)
     (in_bom yes) (on_board yes) (fields_autoplaced)
-    (property "Reference" "#PWR0128" (id 0) (at 88.9 71.12 0)
+    (property "Reference" "#PWR0132" (id 0) (at 88.9 71.12 0)
       (effects (font (size 1.27 1.27)) hide)
     )
@@
   (symbol (lib_id "Connector:Screw_Terminal_01x08") (at 22.225 99.06 0) (mirror y) (unit 1)
     (in_bom yes) (on_board yes) (fields_autoplaced)
-    (property "Reference" "J?" (id 0) (at 22.225 85.09 0))
+    (property "Reference" "J10" (id 0) (at 22.225 85.09 0))
     (property "Value" "Screw_Terminal_01x08" (id 1) (at 22.225 87.63 0))
     (property "Footprint" "IVS_FOOTPRINTS:HT-3.96mm" (id 2) (at 22.225 99.06 0)
@@
   (symbol (lib_id "power:+24V") (at 88.9 156.21 0) (unit 1)
     (in_bom yes) (on_board yes) (fields_autoplaced)
-    (property "Reference" "#PWR0132" (id 0) (at 88.9 160.02 0)
+    (property "Reference" "#PWR0136" (id 0) (at 88.9 160.02 0)
       (effects (font (size 1.27 1.27)) hide)
     )
@@
   (symbol (lib_id "power:+3V3") (at 102.87 27.94 0) (unit 1)
     (in_bom yes) (on_board yes) (fields_autoplaced)
-    (property "Reference" "#PWR0134" (id 0) (at 102.87 31.75 0)
+    (property "Reference" "#PWR0138" (id 0) (at 102.87 31.75 0)
       (effects (font (size 1.27 1.27)) hide)
     )
@@
   (symbol (lib_id "power:+24V") (at 88.9 111.76 0) (unit 1)
     (in_bom yes) (on_board yes) (fields_autoplaced)
-    (property "Reference" "#PWR0130" (id 0) (at 88.9 115.57 0)
+    (property "Reference" "#PWR0134" (id 0) (at 88.9 115.57 0)
       (effects (font (size 1.27 1.27)) hide)
     )
@@
   (symbol (lib_id "power:GND") (at 88.9 189.23 0) (unit 1)
     (in_bom yes) (on_board yes) (fields_autoplaced)
-    (property "Reference" "#PWR0133" (id 0) (at 88.9 195.58 0)
+    (property "Reference" "#PWR0137" (id 0) (at 88.9 195.58 0)
       (effects (font (size 1.27 1.27)) hide)
     )
@@
   (symbol (lib_id "power:GND") (at 110.49 194.31 0) (unit 1)
     (in_bom yes) (on_board yes) (fields_autoplaced)
-    (property "Reference" "#PWR0139" (id 0) (at 110.49 200.66 0)
+    (property "Reference" "#PWR0143" (id 0) (at 110.49 200.66 0)
       (effects (font (size 1.27 1.27)) hide)
     )
@@
   (symbol (lib_id "power:GND") (at 110.49 59.69 0) (unit 1)
     (in_bom yes) (on_board yes) (fields_autoplaced)
-    (property "Reference" "#PWR0136" (id 0) (at 110.49 66.04 0)
+    (property "Reference" "#PWR0140" (id 0) (at 110.49 66.04 0)
       (effects (font (size 1.27 1.27)) hide)
     )
@@
   (symbol (lib_id "power:GND") (at 88.9 54.61 0) (unit 1)
     (in_bom yes) (on_board yes) (fields_autoplaced)
-    (property "Reference" "#PWR0127" (id 0) (at 88.9 60.96 0)
+    (property "Reference" "#PWR0131" (id 0) (at 88.9 60.96 0)
       (effects (font (size 1.27 1.27)) hide)
     )
@@
   (symbol (lib_id "power:+24V") (at 88.9 22.86 0) (unit 1)
     (in_bom yes) (on_board yes) (fields_autoplaced)
-    (property "Reference" "#PWR0126" (id 0) (at 88.9 26.67 0)
+    (property "Reference" "#PWR0130" (id 0) (at 88.9 26.67 0)
       (effects (font (size 1.27 1.27)) hide)
     )
@@
   (symbol (lib_id "power:+3V3") (at 135.89 34.29 0) (unit 1)
     (in_bom yes) (on_board yes) (fields_autoplaced)
-    (property "Reference" "#PWR0141" (id 0) (at 135.89 38.1 0)
+    (property "Reference" "#PWR0145" (id 0) (at 135.89 38.1 0)
       (effects (font (size 1.27 1.27)) hide)
     )
@@
   (symbol (lib_id "power:+3V3") (at 135.89 168.91 0) (unit 1)
     (in_bom yes) (on_board yes) (fields_autoplaced)
-    (property "Reference" "#PWR0144" (id 0) (at 135.89 172.72 0)
-      (effects (font (size 1.27 1.27)) hide)
-    )
+    (property "Reference" "#PWR0148" (id 0) (at 135.89 172.72 0)
+      (effects (font (size 1.27 1.27)) hide)
+    )

Commit message: add shematics MVA
Parts:
- removed R87, R88, R89, R90: 1k, IVS_FOOTPRINTS:R0603, symbol Device:R
Changed lines of the file:
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@@
-    (stroke (width 0) (type default))
-  )
-  (wire (pts (xy 110.49 50.8) (xy 110.49 49.53))
     (stroke (width 0) (type default))
   )
@@
     (stroke (width 0) (type default))
   )
-  (wire (pts (xy 110.49 105.41) (xy 110.49 104.14))
-    (stroke (width 0) (type default))
-  )
   (wire (pts (xy 80.01 26.67) (xy 80.01 22.86))
     (stroke (width 0) (type default))
@@
     (stroke (width 0) (type default))
   )
-  (wire (pts (xy 110.49 185.42) (xy 110.49 184.15))
-    (stroke (width 0) (type default))
-  )
   (wire (pts (xy 74.93 26.67) (xy 80.01 26.67))
     (stroke (width 0) (type default))
@@
     (stroke (width 0) (type default))
   )
-  (wire (pts (xy 110.49 148.59) (xy 110.49 147.32))
-    (stroke (width 0) (type default))
-  )
   (wire (pts (xy 77.47 90.17) (xy 77.47 83.82))
     (stroke (width 0) (type default))
   )
-  (wire (pts (xy 110.49 96.52) (xy 110.49 95.25))
-    (stroke (width 0) (type default))
-  )
   (wire (pts (xy 88.9 68.58) (xy 88.9 69.85))
     (stroke (width 0) (type default))
@@
     (stroke (width 0) (type default))
   )
-  (wire (pts (xy 110.49 59.69) (xy 110.49 58.42))
-    (stroke (width 0) (type default))
-  )
   (wire (pts (xy 73.66 128.27) (xy 77.47 128.27))
     (stroke (width 0) (type default))
@@
     (stroke (width 0) (type default))
   )
-  (wire (pts (xy 110.49 194.31) (xy 110.49 193.04))
-    (stroke (width 0) (type default))
-  )
   (wire (pts (xy 88.9 121.92) (xy 88.9 123.19))
     (stroke (width 0) (type default))
@@
   )
   (wire (pts (xy 102.87 27.94) (xy 105.41 27.94))
-    (stroke (width 0) (type default))
-  )
-  (wire (pts (xy 110.49 139.7) (xy 110.49 138.43))
     (stroke (width 0) (type default))
   )
@@
     )
   )
-  (symbol (lib_id "power:GND") (at 110.49 148.59 0) (unit 1)
-    (in_bom yes) (on_board yes) (dnp no) (fields_autoplaced)
-    (property "Reference" "#PWR0142" (at 110.49 154.94 0)
-      (effects (font (size 1.27 1.27)) hide)
-    )
-    (property "Value" "GND" (at 110.49 153.67 0)
-      (effects (font (size 1.27 1.27)))
-    )
-    (property "Footprint" "" (at 110.49 148.59 0)
-      (effects (font (size 1.27 1.27)) hide)
-    )
-    (property "Datasheet" "" (at 110.49 148.59 0)
-      (effects (font (size 1.27 1.27)) hide)
-    )
-    (pin "1")
-    (instances
-      (project "dongtam"
-        (path "/6833aec4-3d1d-4261-9b3e-f0452b565dd3/992d1183-82f3-4ab3-a77f-7ab8cf195fcd/e4ad1a02-817a-4cce-9ee6-266c75a94756/f9795dc8-b42c-4c97-abd2-37fcb9067069"
-          (reference "#PWR0142") (unit 1)
-        )
-      )
-    )
-  )
   (symbol (lib_id "Device:R") (at 88.9 138.43 0) (unit 1)
     (in_bom yes) (on_board yes) (dnp no)
@@
         (path "/6833aec4-3d1d-4261-9b3e-f0452b565dd3/992d1183-82f3-4ab3-a77f-7ab8cf195fcd/e4ad1a02-817a-4cce-9ee6-266c75a94756/f9795dc8-b42c-4c97-abd2-37fcb9067069"
           (reference "D21") (unit 1)
-        )
-      )
-    )
-  )
-  (symbol (lib_id "power:GND") (at 110.49 105.41 0) (unit 1)
-    (in_bom yes) (on_board yes) (dnp no) (fields_autoplaced)
-    (property "Reference" "#PWR0141" (at 110.49 111.76 0)
-      (effects (font (size 1.27 1.27)) hide)
-    )
-    (property "Value" "GND" (at 110.49 110.49 0)
-      (effects (font (size 1.27 1.27)))
-    )
-    (property "Footprint" "" (at 110.49 105.41 0)
-      (effects (font (size 1.27 1.27)) hide)
-    )
-    (property "Datasheet" "" (at 110.49 105.41 0)
-      (effects (font (size 1.27 1.27)) hide)
-    )
-    (pin "1")
-    (instances
-      (project "dongtam"
-        (path "/6833aec4-3d1d-4261-9b3e-f0452b565dd3/992d1183-82f3-4ab3-a77f-7ab8cf195fcd/e4ad1a02-817a-4cce-9ee6-266c75a94756/f9795dc8-b42c-4c97-abd2-37fcb9067069"
-          (reference "#PWR0141") (unit 1)
         )
       )
@@
     )
   )
-  (symbol (lib_id "Device:R") (at 110.49 100.33 0) (unit 1)
-    (in_bom yes) (on_board yes) (dnp no)
-    (property "Reference" "R88" (at 111.76 99.06 0)
-      (effects (font (size 1.27 1.27)) (justify left))
-    )
-    (property "Value" "1k" (at 111.76 101.6 0)
-      (effects (font (size 1.27 1.27)) (justify left))
-    )
-    (property "Footprint" "IVS_FOOTPRINTS:R0603" (at 108.712 100.33 90)
-      (effects (font (size 1.27 1.27)) hide)
-    )
-    (property "Datasheet" "~" (at 110.49 100.33 0)
-      (effects (font (size 1.27 1.27)) hide)
-    )
-    (pin "1")
-    (pin "2")
-    (instances
-      (project "dongtam"
-        (path "/6833aec4-3d1d-4261-9b3e-f0452b565dd3/992d1183-82f3-4ab3-a77f-7ab8cf195fcd/e4ad1a02-817a-4cce-9ee6-266c75a94756/f9795dc8-b42c-4c97-abd2-37fcb9067069"
-          (reference "R88") (unit 1)
-        )
-      )
-    )
-  )
   (symbol (lib_id "Connector:Screw_Terminal_01x08") (at 22.225 99.06 0) (mirror y) (unit 1)
     (in_bom yes) (on_board yes) (dnp no) (fields_autoplaced)
@@
     )
   )
-  (symbol (lib_id "Device:R") (at 110.49 143.51 0) (unit 1)
-    (in_bom yes) (on_board yes) (dnp no)
-    (property "Reference" "R89" (at 111.76 142.24 0)
-      (effects (font (size 1.27 1.27)) (justify left))
-    )
-    (property "Value" "1k" (at 111.76 144.78 0)
-      (effects (font (size 1.27 1.27)) (justify left))
-    )
-    (property "Footprint" "IVS_FOOTPRINTS:R0603" (at 108.712 143.51 90)
-      (effects (font (size 1.27 1.27)) hide)
-    )
-    (property "Datasheet" "~" (at 110.49 143.51 0)
-      (effects (font (size 1.27 1.27)) hide)
-    )
-    (pin "1")
-    (pin "2")
-    (instances
-      (project "dongtam"
-        (path "/6833aec4-3d1d-4261-9b3e-f0452b565dd3/992d1183-82f3-4ab3-a77f-7ab8cf195fcd/e4ad1a02-817a-4cce-9ee6-266c75a94756/f9795dc8-b42c-4c97-abd2-37fcb9067069"
-          (reference "R89") (unit 1)
-        )
-      )
-    )
-  )
   (symbol (lib_id "Device:R") (at 135.89 173.99 0) (unit 1)
     (in_bom yes) (on_board yes) (dnp no)
@@
         (path "/6833aec4-3d1d-4261-9b3e-f0452b565dd3/992d1183-82f3-4ab3-a77f-7ab8cf195fcd/e4ad1a02-817a-4cce-9ee6-266c75a94756/f9795dc8-b42c-4c97-abd2-37fcb9067069"
           (reference "R94") (unit 1)
-        )
-      )
-    )
-  )
-  (symbol (lib_id "Device:R") (at 110.49 54.61 0) (unit 1)
-    (in_bom yes) (on_board yes) (dnp no)
-    (property "Reference" "R87" (at 111.76 53.34 0)
-      (effects (font (size 1.27 1.27)) (justify left))
-    )
-    (property "Value" "1k" (at 111.76 55.88 0)
-      (effects (font (size 1.27 1.27)) (justify left))
-    )
-    (property "Footprint" "IVS_FOOTPRINTS:R0603" (at 108.712 54.61 90)
-      (effects (font (size 1.27 1.27)) hide)
-    )
-    (property "Datasheet" "~" (at 110.49 54.61 0)
-      (effects (font (size 1.27 1.27)) hide)
-    )
-    (pin "1")
-    (pin "2")
-    (instances
-      (project "dongtam"
-        (path "/6833aec4-3d1d-4261-9b3e-f0452b565dd3/992d1183-82f3-4ab3-a77f-7ab8cf195fcd/e4ad1a02-817a-4cce-9ee6-266c75a94756/f9795dc8-b42c-4c97-abd2-37fcb9067069"
-          (reference "R87") (unit 1)
         )
       )
@@
     )
   )
-  (symbol (lib_id "Device:R") (at 110.49 189.23 0) (unit 1)
-    (in_bom yes) (on_board yes) (dnp no)
-    (property "Reference" "R90" (at 111.76 187.96 0)
-      (effects (font (size 1.27 1.27)) (justify left))
-    )
-    (property "Value" "1k" (at 111.76 190.5 0)
-      (effects (font (size 1.27 1.27)) (justify left))
-    )
-    (property "Footprint" "IVS_FOOTPRINTS:R0603" (at 108.712 189.23 90)
-      (effects (font (size 1.27 1.27)) hide)
-    )
-    (property "Datasheet" "~" (at 110.49 189.23 0)
-      (effects (font (size 1.27 1.27)) hide)
-    )
-    (pin "1")
-    (pin "2")
-    (instances
-      (project "dongtam"
-        (path "/6833aec4-3d1d-4261-9b3e-f0452b565dd3/992d1183-82f3-4ab3-a77f-7ab8cf195fcd/e4ad1a02-817a-4cce-9ee6-266c75a94756/f9795dc8-b42c-4c97-abd2-37fcb9067069"
-          (reference "R90") (unit 1)
-        )
-      )
-    )
-  )
   (symbol (lib_id "Amplifier_Operational:TL084") (at 120.65 181.61 0) (unit 4)
     (in_bom yes) (on_board yes) (dnp no)
@@
         )
       )
-    )
-  )
-  (symbol (lib_id "power:GND") (at 110.49 194.31 0) (unit 1)
-    (in_bom yes) (on_board yes) (dnp no) (fields_autoplaced)
-    (property "Reference" "#PWR0143" (at 110.49 200.66 0)
-      (effects (font (size 1.27 1.27)) hide)
-    )
-    (property "Value" "GND" (at 110.49 199.39 0)
-      (effects (font (size 1.27 1.27)))
-    )
-    (property "Footprint" "" (at 110.49 194.31 0)
-      (effects (font (size 1.27 1.27)) hide)
-    )
-    (property "Datasheet" "" (at 110.49 194.31 0)
-      (effects (font (size 1.27 1.27)) hide)
-    )
-    (pin "1")
-    (instances
-      (project "dongtam"
-        (path "/6833aec4-3d1d-4261-9b3e-f0452b565dd3/992d1183-82f3-4ab3-a77f-7ab8cf195fcd/e4ad1a02-817a-4cce-9ee6-266c75a94756/f9795dc8-b42c-4c97-abd2-37fcb9067069"
-          (reference "#PWR0143") (unit 1)
-        )
-      )
-    )
-  )
-  (symbol (lib_id "power:GND") (at 110.49 59.69 0) (unit 1)
-    (in_bom yes) (on_board yes) (dnp no) (fields_autoplaced)
-    (property "Reference" "#PWR0140" (at 110.49 66.04 0)
-      (effects (font (size 1.27 1.27)) hide)
-    )
-    (property "Value" "GND" (at 110.49 64.77 0)
-      (effects (font (size 1.27 1.27)))
-    )
-    (property "Footprint" "" (at 110.49 59.69 0)
-      (effects (font (size 1.27 1.27)) hide)
-    )
-    (property "Datasheet" "" (at 110.49 59.69 0)
-      (effects (font (size 1.27 1.27)) hide)
-    )
-    (pin "1")
-    (instances
-      (project "dongtam"
-        (path "/6833aec4-3d1d-4261-9b3e-f0452b565dd3/992d1183-82f3-4ab3-a77f-7ab8cf195fcd/e4ad1a02-817a-4cce-9ee6-266c75a94756/f9795dc8-b42c-4c97-abd2-37fcb9067069"
-          (reference "#PWR0140") (unit 1)
-        )
-      )

Commit message: layout PCB part 1
Parts:
- removed Q13, Q14, Q15, Q16: SI_2300, IVS_FOOTPRINTS:SOT23-3, symbol Device:Q_NMOS_DGS
- added Q12, Q13, Q14, Q15: N_Mosfet, IVS_FOOTPRINTS:SOT23-3, symbol IVS_SYMBOLS:N_Mosfet
Connections:
- net VAN13-: now also J10.8 (Pin_8), Q12.3 (D); no longer J10.2 (Pin_2)
- net VAN13_input: now also Q12.1 (G)
- net VAN14-: now also J10.6 (Pin_6), Q13.3 (D); no longer J10.4 (Pin_4)
- net VAN14_input: now also Q13.1 (G)
- net VAN15-: now also J10.4 (Pin_4), Q14.3 (D); no longer J10.6 (Pin_6)
- net VAN15_input: now also Q14.1 (G)
- net VAN16-: now also J10.2 (Pin_2), Q15.3 (D); no longer J10.8 (Pin_8)
- net VAN16_input: now also Q15.1 (G)
- net at R86.1, U14.12 (+): now also Q15.2 (S)
- net at R83.1, U14.3 (+): now also Q12.2 (S)
- net at R84.1, U14.5 (+): now also Q13.2 (S)
- net at R85.1, U14.10 (+): now also Q14.2 (S)
